File: extended/xfm2.sch (KiCad schematic (older format))
At the start: 23 parts, among them J1 Midi In, J2 Pin Breakout, J3 Midi Out, J4 Midi Thru, J5 Conn_Coaxial, U1 4N36, U2 CmodA7-35T, U3 24LC01, U4 UDA1334A

Commit message: updated schematic
Parts:
- removed U1: 4N36, Package_DIP:SMDIP-6_W9.53mm_Clearance8mm, symbol Isolator:4N36
- added FB1, FB2, FB3, FB4, FB5, FB6: Ferrite_Bead, Capacitor_SMD:C_0805_2012Metric_Pad1.18x1.45mm_HandSolder, symbol Device:Ferrite_Bead
- added R10, R9: 10, Resistor_SMD:R_0805_2012Metric_Pad1.20x1.40mm_HandSolder, symbol Device:R
- added U1: H11L1, Package_DIP:SMDIP-6_W9.53mm_Clearance8mm, symbol Isolator:H11L1
- added U5: 74HC14, Package_SO:SO-14_3.9x8.65mm_P1.27mm, symbol 74xx:74HC14
- D1: footprint samacsys:SODFL1608X70N -> Diode_SMD:D_SOD-523
- D2: value LED_MIDI_1 -> LED_MIDI_IN
- D3: value LED_MIDI_2 -> LED_MIDI_OUT
- R5, R6, R7, R8: value 220 -> 2k
Connections:
- net labels added: MIDI_IN_INV
- net labels removed: LED_MIDI_1, LED_MIDI_2, MIDI_IN_RETURN, MIDI_THRU
- wire segments 107 -> 104
- no-connect marks 48 -> 56
Other:
- moved on the sheet: C1, D1, D2, D3, J1, J2, J3, J4, J5, R1, R2, R3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

Commit message: nicer schematic, control voltage, power supply, power cleanups
Parts:
- added C2, C3: 10uF, symbol Device:C
- added C4, C5: 100uF, symbol Device:C
- added C6, C7: 330p-560p, symbol Device:C
- added D6: 1N4002, symbol Device:D
- added J6: Jack-DC, symbol Connector:Jack-DC
- added J7: A-100_Bus_Connector, symbol xfm2:A-100_Bus_Connector
- added J8, J9: AudioJack2, symbol Connector:AudioJack2
- added R11, R12, R13, R14: 100k, symbol Device:R
- added R15, R16: 33k, symbol Device:R
- added R17, R18: 100, symbol Device:R
- added U6: LM1117-5.0, symbol Regulator_Linear:LM1117-5.0
- added U7: LM1117-3.3, symbol Regulator_Linear:LM1117-3.3
- added U8: MCP6004, symbol Amplifier_Operational:MCP6004
- added U9: L7905, symbol Regulator_Linear:L7905
Connections:
- net labels added: +12V, +3.3V, +5V, -12V, -5V, CV0_3.3V, CV1_3.3V
- net labels removed: EEPROM_VCC, I2S_VCC, VCC
- wire segments 104 -> 150
- no-connect marks 56 -> 64
Other:
- note added: "9V-\n12V"
- note added: "Analog Output"
- note added: "Control Voltage"
- note added: "DC Barrel Jack"
- note added: "Digital Output"
- note added: "Eurorack\nA-100"
- note added: "FPGA / Synth"
- note added: "Inputs"
- note added: "LEDs"
- note added: "Memory"
- note added: "Midi Buffer"
- note added: "Midi In"
- note added: "Midi Out"
- note added: "Midi Thru"
- note added: "Outputs"
- note added: "Pin Breakout"
- note added: "Power"
- moved on the sheet: C1, D1, D2, D3, D4, D5, FB1, FB2, FB3, FB4, FB5, FB6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

Commit message: initial extended pcb 1.1 placement
Parts:
- removed C4, C5: 100uF, symbol Device:C
- removed U9: L7905, symbol Regulator_Linear:L7905
- added C4, C5: 100uF, Capacitor_SMD:CP_Elec_6.3x5.7, symbol Device:CP1
- added U9: MC79M05_TO252, Package_TO_SOT_SMD:TO-252-2, symbol Regulator_Linear:MC79M05_TO252
- C2, C3, C6, C7: footprint (none) -> Capacitor_SMD:C_0805_2012Metric_Pad1.18x1.45mm_HandSolder
- D6: value 1N4002 -> 1N4007; footprint (none) -> Diode_SMD:D_MELF_Handsoldering
- J6: footprint (none) -> Connector_BarrelJack:BarrelJack_Wuerth_6941xx301002
- J7: footprint (none) -> Connector_PinHeader_2.54mm:PinHeader_2x08_P2.54mm_Vertical
- J8, J9: footprint (none) -> Connector_Audio:Jack_6.35mm_Neutrik_NRJ6HM-1_Horizontal
- R11, R12, R13, R14, R15, R16, R17, R18: footprint (none) -> Resistor_SMD:R_0805_2012Metric_Pad1.20x1.40mm_HandSolder
- U6, U7: footprint (none) -> Package_TO_SOT_SMD:SOT-223-3_TabPin2
- U8: footprint (none) -> Package_SO:SO-14_5.3x10.2mm_P1.27mm
Changed lines of the file:
@@
 F 0 "J6" H 2900 6750 50  0000 C CNN
 F 1 "Jack-DC" H 2900 6650 50  0000 C CNN
-F 2 "" H 3000 6410 50  0001 C CNN
+F 2 "Connector_BarrelJack:BarrelJack_Wuerth_6941xx301002" H 3000 6410 50  0001 C CNN
 F 3 "~" H 3000 6410 50  0001 C CNN
 	1    2950 6450
@@
 Wire Notes Line
 	2700 4350 5400 4350
-Connection ~ 4750 7150
-Wire Wire Line
-	4750 7150 5000 7150
-Connection ~ 4750 6350
-Wire Wire Line
-	4750 6350 5000 6350
 $Comp
 L power:+3.3V #PWR0137
@@
 	1    0    0    -1
 $EndComp
-Wire Wire Line
-	4650 6350 4750 6350
-Wire Wire Line
-	4650 7150 4750 7150
 $Comp
 L power:GND #PWR0131
@@
 F 0 "U6" H 4350 6592 50  0000 C CNN
 F 1 "LM1117-5.0" H 4350 6501 50  0000 C CNN
-F 2 "" H 4350 6350 50  0001 C CNN
+F 2 "Package_TO_SOT_SMD:SOT-223-3_TabPin2" H 4350 6350 50  0001 C CNN
 F 3 "http://www.ti.com/lit/ds/symlink/lm1117.pdf" H 4350 6350 50  0001 C CNN
 	1    4350 6350
@@
 F 0 "U7" H 4150 7300 50  0000 C CNN
 F 1 "LM1117-3.3" H 4500 7300 50  0000 C CNN
-F 2 "" H 4350 7150 50  0001 C CNN
+F 2 "Package_TO_SOT_SMD:SOT-223-3_TabPin2" H 4350 7150 50  0001 C CNN
 F 3 "http://www.ti.com/lit/ds/symlink/lm1117.pdf" H 4350 7150 50  0001 C CNN
 	1    4350 7150
@@
 F 0 "J7" H 3600 6025 50  0000 C CNN
 F 1 "A-100_Bus_Connector" H 3600 5934 50  0000 C CNN
-F 2 "" H 3400 5500 50  0001 C CNN
+F 2 "Connector_PinHeader_2.54mm:PinHeader_2x08_P2.54mm_Vertical" H 3400 5500 50  0001 C CNN
 F 3 "~" H 3400 5500 50  0001 C CNN
 	1    3550 5500
@@
 P 3450 6350
 F 0 "D6" H 3450 6550 50  0000 C CNN
-F 1 "1N4002" H 3450 6450 50  0000 C CNN
-F 2 "" H 3450 6350 50  0001 C CNN
+F 1 "1N4007" H 3450 6450 50  0000 C CNN
+F 2 "Diode_SMD:D_MELF_Handsoldering" H 3450 6350 50  0001 C CNN
 F 3 "~" H 3450 6350 50  0001 C CNN
 	1    3450 6350
 	-1   0    0    1
-$EndComp
-$Comp
-L Device:C C5
-U 1 1 61280FAF
-P 4750 7300
-F 0 "C5" H 4865 7346 50  0000 L CNN
-F 1 "100uF" H 4865 7255 50  0000 L CNN
-F 2 "" H 4788 7150 50  0001 C CNN
-F 3 "~" H 4750 7300 50  0001 C CNN
-	1    4750 7300
-	1    0    0    -1
-$EndComp
-$Comp
-L Device:C C4
-U 1 1 612812C3
-P 4750 6500
-F 0 "C4" H 4865 6546 50  0000 L CNN
-F 1 "100uF" H 4865 6455 50  0000 L CNN
-F 2 "" H 4788 6350 50  0001 C CNN
-F 3 "~" H 4750 6500 50  0001 C CNN
-	1    4750 6500
-	1    0    0    -1
 $EndComp
 $Comp
@@
 F 0 "C2" H 3865 7346 50  0000 L CNN
 F 1 "10uF" H 3865 7255 50  0000 L CNN
-F 2 "" H 3788 7150 50  0001 C CNN
+F 2 "Capacitor_SMD:C_0805_2012Metric_Pad1.18x1.45mm_HandSolder" H 3788 7150 50  0001 C CNN
 F 3 "~" H 3750 7300 50  0001 C CNN
 	1    3750 7300
@@
 F 0 "C3" H 3915 6546 50  0000 L CNN
 F 1 "10uF" H 3915 6455 50  0000 L CNN
-F 2 "" H 3838 6350 50  0001 C CNN
+F 2 "Capacitor_SMD:C_0805_2012Metric_Pad1.18x1.45mm_HandSolder" H 3838 6350 50  0001 C CNN
 F 3 "~" H 3800 6500 50  0001 C CNN
 	1    3800 6500
@@
 F 0 "R15" V 2643 2600 50  0000 C CNN
 F 1 "33k" V 2734 2600 50  0000 C CNN
-F 2 "" V 2780 2600 50  0001 C CNN
+F 2 "Resistor_SMD:R_0805_2012Metric_Pad1.20x1.40mm_HandSolder" V 2780 2600 50  0001 C CNN
 F 3 "~" H 2850 2600 50  0001 C CNN
 	1    2850 2600
@@
 F 0 "R17" V 3557 2250 50  0000 C CNN
 F 1 "100" V 3466 2250 50  0000 C CNN
-F 2 "" V 3280 2250 50  0001 C CNN
+F 2 "Resistor_SMD:R_0805_2012Metric_Pad1.20x1.40mm_HandSolder" V 3280 2250 50  0001 C CNN
 F 3 "~" H 3350 2250 50  0001 C CNN
 	1    3350 2250
@@
 F 0 "U8" H 858 3096 50  0000 L CNN
 F 1 "MCP6004" H 858 3005 50  0000 L CNN
-F 2 "" H 850 3150 50  0001 C CNN
+F 2 "Package_SO:SO-14_5.3x10.2mm_P1.27mm" H 850 3150 50  0001 C CNN
 F 3 "http://ww1.microchip.com/downloads/en/DeviceDoc/21733j.pdf" H 950 3250 50  0001 C CNN
 	5    900  3050
@@
 F 0 "J8" H 1532 2775 50  0000 C CNN
 F 1 "AudioJack2" H 1532 2684 50  0000 C CNN
-F 2 "" H 1500 2450 50  0001 C CNN
+F 2 "Connector_Audio:Jack_6.35mm_Neutrik_NRJ6HM-1_Horizontal" H 1500 2450 50  0001 C CNN
 F 3 "~" H 1500 2450 50  0001 C CNN
 	1    1500 2450
@@
 F 0 "U8" H 4550 3817 50  0000 C CNN
 F 1 "MCP6004" H 4550 3726 50  0000 C CNN
-F 2 "" H 4500 3550 50  0001 C CNN
+F 2 "Package_SO:SO-14_5.3x10.2mm_P1.27mm" H 4500 3550 50  0001 C CNN
 F 3 "http://ww1.microchip.com/downloads/en/DeviceDoc/21733j.pdf" H 4600 3650 50  0001 C CNN
 	4    4550 3450
@@
 F 0 "U8" H 4550 2617 50  0000 C CNN
 F 1 "MCP6004" H 4550 2526 50  0000 C CNN
-F 2 "" H 4500 2350 50  0001 C CNN
+F 2 "Package_SO:SO-14_5.3x10.2mm_P1.27mm" H 4500 2350 50  0001 C CNN
 F 3 "http://ww1.microchip.com/downloads/en/DeviceDoc/21733j.pdf" H 4600 2450 50  0001 C CNN
 	3    4550 2250
@@
 F 0 "R11" V 1693 2350 50  0000 C CNN
 F 1 "100k" V 1784 2350 50  0000 C CNN
-F 2 "" V 1830 2350 50  0001 C CNN
+F 2 "Resistor_SMD:R_0805_2012Metric_Pad1.20x1.40mm_HandSolder" V 1830 2350 50  0001 C CNN
 F 3 "~" H 1900 2350 50  0001 C CNN
 	1    1900 2350
@@
 F 0 "R13" H 2030 2054 50  0000 R CNN
 F 1 "100k" H 2030 2145 50  0000 R CNN
-F 2 "" V 2030 2100 50  0001 C CNN
+F 2 "Resistor_SMD:R_0805_2012Metric_Pad1.20x1.40mm_HandSolder" V 2030 2100 50  0001 C CNN
 F 3 "~" H 2100 2100 50  0001 C CNN
 	1    2100 2100
@@
 F 0 "U8" H 2800 2617 50  0000 C CNN
 F 1 "MCP6004" H 2800 2526 50  0000 C CNN
-F 2 "" H 2750 2350 50  0001 C CNN
+F 2 "Package_SO:SO-14_5.3x10.2mm_P1.27mm" H 2750 2350 50  0001 C CNN
 F 3 "http://ww1.microchip.com/downloads/en/DeviceDoc/21733j.pdf" H 2850 2450 50  0001 C CNN
 	1    2800 2250
@@
 F 0 "U8" H 2800 3867 50  0000 C CNN
 F 1 "MCP6004" H 2800 3776 50  0000 C CNN
-F 2 "" H 2750 3600 50  0001 C CNN
+F 2 "Package_SO:SO-14_5.3x10.2mm_P1.27mm" H 2750 3600 50  0001 C CNN
 F 3 "http://ww1.microchip.com/downloads/en/DeviceDoc/21733j.pdf" H 2850 3700 50  0001 C CNN
 	2    2800 3500
@@
 F 0 "C6" V 2548 2950 50  0000 C CNN
 F 1 "330p-560p" V 2639 2950 50  0000 C CNN
-F 2 "" H 2838 2800 50  0001 C CNN
+F 2 "Capacitor_SMD:C_0805_2012Metric_Pad1.18x1.45mm_HandSolder" H 2838 2800 50  0001 C CNN
 F 3 "~" H 2800 2950 50  0001 C CNN
 	1    2800 2950
@@
 F 0 "J9" H 1532 4025 50  0000 C CNN
 F 1 "AudioJack2" H 1532 3934 50  0000 C CNN
-F 2 "" H 1500 3700 50  0001 C CNN
+F 2 "Connector_Audio:Jack_6.35mm_Neutrik_NRJ6HM-1_Horizontal" H 1500 3700 50  0001 C CNN
 F 3 "~" H 1500 3700 50  0001 C CNN
 	1    1500 3700
@@
 F 0 "R12" V 1693 3600 50  0000 C CNN
 F 1 "100k" V 1784 3600 50  0000 C CNN
-F 2 "" V 1830 3600 50  0001 C CNN
+F 2 "Resistor_SMD:R_0805_2012Metric_Pad1.20x1.40mm_HandSolder" V 1830 3600 50  0001 C CNN
 F 3 "~" H 1900 3600 50  0001 C CNN
 	1    1900 3600
@@
 F 0 "R14" H 2030 3304 50  0000 R CNN
 F 1 "100k" H 2030 3395 50  0000 R CNN
-F 2 "" V 2030 3350 50  0001 C CNN
+F 2 "Resistor_SMD:R_0805_2012Metric_Pad1.20x1.40mm_HandSolder" V 2030 3350 50  0001 C CNN
 F 3 "~" H 2100 3350 50  0001 C CNN
 	1    2100 3350
@@
 F 0 "R18" V 3557 3500 50  0000 C CNN
 F 1 "100" V 3466 3500 50  0000 C CNN
-F 2 "" V 3280 3500 50  0001 C CNN
+F 2 "Resistor_SMD:R_0805_2012Metric_Pad1.20x1.40mm_HandSolder" V 3280 3500 50  0001 C CNN
 F 3 "~" H 3350 3500 50  0001 C CNN
 	1    3350 3500
@@
 F 0 "R16" V 2643 3850 50  0000 C CNN
 F 1 "33k" V 2734 3850 50  0000 C CNN
-F 2 "" V 2780 3850 50  0001 C CNN
+F 2 "Resistor_SMD:R_0805_2012Metric_Pad1.20x1.40mm_HandSolder" V 2780 3850 50  0001 C CNN
 F 3 "~" H 2850 3850 50  0001 C CNN
 	1    2850 3850
@@
 F 0 "C7" V 2950 4250 50  0000 C CNN
 F 1 "330p-560p" V 2689 4150 50  0000 C CNN
-F 2 "" H 2888 4000 50  0001 C CNN
+F 2 "Capacitor_SMD:C_0805_2012Metric_Pad1.18x1.45mm_HandSolder" H 2888 4000 50  0001 C CNN
 F 3 "~" H 2850 4150 50  0001 C CNN
 	1    2850 4150
@@
 $EndComp
 $Comp
-L Regulator_Linear:L7905 U9
-U 1 1 61F85494
-P 4850 5600
-F 0 "U9" H 4850 5451 50  0000 C CNN
-F 1 "L7905" H 4850 5360 50  0000 C CNN
-F 2 "" H 4850 5400 50  0001 C CIN
-F 3 "http://www.st.com/content/ccc/resource/technical/document/datasheet/c9/16/86/41/c7/2b/45/f2/CD00000450.pdf/files/CD00000450.pdf/jcr:content/translations/en.CD00000450.pdf" H 4850 5600 50  0001 C CNN
-	1    4850 5600
-	1    0    0    -1
-$EndComp
-$Comp
 L power:-5V #PWR012
 U 1 1 62061E3F
@@
 $EndComp
 NoConn ~ 7650 5850
+$Comp
+L Device:CP1 C4
+U 1 1 620B53AC
+P 4750 6500
+F 0 "C4" H 4865 6546 50  0000 L CNN
+F 1 "100uF" H 4865 6455 50  0000 L CNN
+F 2 "Capacitor_SMD:CP_Elec_6.3x5.7" H 4750 6500 50  0001 C CNN
+F 3 "~" H 4750 6500 50  0001 C CNN
+	1    4750 6500
+	1    0    0    -1
+$EndComp
+$Comp
+L Device:CP1 C5
+U 1 1 620B6A88
+P 4750 7300
+F 0 "C5" H 4865 7346 50  0000 L CNN
+F 1 "100uF" H 4865 7255 50  0000 L CNN
+F 2 "Capacitor_SMD:CP_Elec_6.3x5.7" H 4750 7300 50  0001 C CNN
+F 3 "~" H 4750 7300 50  0001 C CNN
+	1    4750 7300
+	1    0    0    -1
+$EndComp
+Wire Wire Line
+	4650 7150 4750 7150
+Connection ~ 4750 7150
+Wire Wire Line
+	4750 7150 5000 7150
+Wire Wire Line
+	4650 6350 4750 6350
+Connection ~ 4750 6350
+Wire Wire Line
+	4750 6350 5000 6350
+$Comp
+L Regulator_Linear:MC79M05_TO252 U9
+U 1 1 6216B584
+P 4850 5600
+F 0 "U9" H 4850 5451 50  0000 C CNN
+F 1 "MC79M05_TO252" H 4850 5360 50  0000 C CNN
+F 2 "Package_TO_SOT_SMD:TO-252-2" H 4850 5400 50  0001 C CIN
+F 3 "http://www.onsemi.com/pub/Collateral/MC79M00-D.PDF" H 4850 5600 50  0001 C CNN
+	1    4850 5600
+	1    0    0    -1
+$EndComp
 $EndSCHEMATC

Commit message: fixes
Parts:
- D1: footprint Diode_SMD:D_SOD-523 -> Diode_SMD:D_SOD-323_HandSoldering
Changed lines of the file:
@@
 F 0 "D1" H 2900 1567 50  0000 C CNN
 F 1 "D" H 2900 1476 50  0000 C CNN
-F 2 "Diode_SMD:D_SOD-523" H 2900 1350 50  0001 C CNN
+F 2 "Diode_SMD:D_SOD-323_HandSoldering" H 2900 1350 50  0001 C CNN
 F 3 "~" H 2900 1350 50  0001 C CNN
 	1    2900 1350

Commit message: power updates.
Parts:
- removed U9: MC79M05_TO252, Package_TO_SOT_SMD:TO-252-2, symbol Regulator_Linear:MC79M05_TO252
- added C8: 0.33uF, Capacitor_Tantalum_SMD:CP_EIA-3216-18_Kemet-A_Pad1.58x1.35mm_HandSolder, symbol Device:CP1
- added C9: 0.1uF, Capacitor_Tantalum_SMD:CP_EIA-3216-18_Kemet-A_Pad1.58x1.35mm_HandSolder, symbol Device:CP1
- added U9: L79L05_SO8, Package_SO:SOIC-8_3.9x4.9mm_P1.27mm, symbol Regulator_Linear:L79L05_SO8
- C4, C5: value 100uF -> 10uF; footprint Capacitor_SMD:CP_Elec_6.3x5.7 -> Capacitor_Tantalum_SMD:CP_EIA-3216-18_Kemet-A_Pad1.58x1.35mm_HandSolder
Connections:
- net -12V: now also C8.1, U9.2 (IN), U9.3 (IN), U9.6 (IN), U9.7 (IN)
- net -5V: now also C9.1, U9.1 (OUT)
- net GND: now also C8.2, C9.2, U9.5 (GND)
Changed lines of the file:
@@
 	6550 4750 6550 4850
 Wire Wire Line
-	4500 5550 4500 5600
+	4500 5450 4500 5500
 Wire Wire Line
-	4500 5600 4550 5600
+	4500 5500 4550 5500
 Wire Wire Line
-	4850 5300 4850 5250
+	4850 5200 4850 5150
 $Comp
 L power:GND #PWR011
 U 1 1 61FB0BB8
-P 4850 5250
-F 0 "#PWR011" H 4850 5000 50  0001 C CNN
-F 1 "GND" V 4855 5122 50  0000 R CNN
-F 2 "" H 4850 5250 50  0001 C CNN
-F 3 "" H 4850 5250 50  0001 C CNN
-	1    4850 5250
+P 4850 5150
+F 0 "#PWR011" H 4850 4900 50  0001 C CNN
+F 1 "GND" V 4855 5022 50  0000 R CNN
+F 2 "" H 4850 5150 50  0001 C CNN
+F 3 "" H 4850 5150 50  0001 C CNN
+	1    4850 5150
 	-1   0    0    1
 $EndComp
@@
 L power:-12V #PWR010
 U 1 1 61FB0352
-P 4500 5550
-F 0 "#PWR010" H 4500 5650 50  0001 C CNN
-F 1 "-12V" H 4515 5723 50  0000 C CNN
-F 2 "" H 4500 5550 50  0001 C CNN
-F 3 "" H 4500 5550 50  0001 C CNN
-	1    4500 5550
+P 4500 5450
+F 0 "#PWR010" H 4500 5550 50  0001 C CNN
+F 1 "-12V" H 4515 5623 50  0000 C CNN
+F 2 "" H 4500 5450 50  0001 C CNN
+F 3 "" H 4500 5450 50  0001 C CNN
+	1    4500 5450
 	1    0    0    -1
 $EndComp
@@
 L power:-5V #PWR012
 U 1 1 62061E3F
-P 5200 5550
-F 0 "#PWR012" H 5200 5650 50  0001 C CNN
-F 1 "-5V" H 5215 5723 50  0000 C CNN
-F 2 "" H 5200 5550 50  0001 C CNN
-F 3 "" H 5200 5550 50  0001 C CNN
-	1    5200 5550
+P 5200 5450
+F 0 "#PWR012" H 5200 5550 50  0001 C CNN
+F 1 "-5V" H 5215 5623 50  0000 C CNN
+F 2 "" H 5200 5450 50  0001 C CNN
+F 3 "" H 5200 5450 50  0001 C CNN
+	1    5200 5450
 	1    0    0    -1
 $EndComp
 Wire Wire Line
-	5150 5600 5200 5600
-Wire Wire Line
-	5200 5600 5200 5550
+	5200 5500 5200 5450
 $Comp
 L power:+3.3V #PWR0116
@@
 $EndComp
 NoConn ~ 7650 5850
+Wire Wire Line
+	4750 7150 5000 7150
+Wire Wire Line
+	4650 7150 4750 7150
+Connection ~ 4750 7150
+$Comp
+L Device:CP1 C5
+U 1 1 620B6A88
+P 4750 7300
+F 0 "C5" H 4865 7346 50  0000 L CNN
+F 1 "10uF" H 4865 7255 50  0000 L CNN
+F 2 "Capacitor_Tantalum_SMD:CP_EIA-3216-18_Kemet-A_Pad1.58x1.35mm_HandSolder" H 4750 7300 50  0001 C CNN
+F 3 "~" H 4750 7300 50  0001 C CNN
+	1    4750 7300
+	1    0    0    -1
+$EndComp
+Wire Wire Line
+	4750 6350 5000 6350
+Wire Wire Line
+	4650 6350 4750 6350
+Connection ~ 4750 6350
 $Comp
 L Device:CP1 C4
@@
 P 4750 6500
 F 0 "C4" H 4865 6546 50  0000 L CNN
-F 1 "100uF" H 4865 6455 50  0000 L CNN
-F 2 "Capacitor_SMD:CP_Elec_6.3x5.7" H 4750 6500 50  0001 C CNN
+F 1 "10uF" H 4865 6455 50  0000 L CNN
+F 2 "Capacitor_Tantalum_SMD:CP_EIA-3216-18_Kemet-A_Pad1.58x1.35mm_HandSolder" H 4750 6500 50  0001 C CNN
 F 3 "~" H 4750 6500 50  0001 C CNN
 	1    4750 6500
@@
 $EndComp
 $Comp
-L Device:CP1 C5
-U 1 1 620B6A88
-P 4750 7300
-F 0 "C5" H 4865 7346 50  0000 L CNN
-F 1 "100uF" H 4865 7255 50  0000 L CNN
-F 2 "Capacitor_SMD:CP_Elec_6.3x5.7" H 4750 7300 50  0001 C CNN
-F 3 "~" H 4750 7300 50  0001 C CNN
-	1    4750 7300
+L Regulator_Linear:L79L05_SO8 U9
+U 1 1 60E73B7F
+P 4850 5500
+F 0 "U9" H 4950 5750 50  0000 C CNN
+F 1 "L79L05_SO8" H 4850 5850 50  0000 C CNN
+F 2 "Package_SO:SOIC-8_3.9x4.9mm_P1.27mm" H 4850 5300 50  0001 C CIN
+F 3 "http://www.farnell.com/datasheets/1827870.pdf" H 4850 5550 50  0001 C CNN
+	1    4850 5500
+	1    0    0    -1
+$EndComp
+$Comp
+L power:GND #PWR0155
+U 1 1 60E82DF4
+P 4500 5800
+F 0 "#PWR0155" H 4500 5550 50  0001 C CNN
+F 1 "GND" V 4505 5672 50  0000 R CNN
+F 2 "" H 4500 5800 50  0001 C CNN
+F 3 "" H 4500 5800 50  0001 C CNN
+	1    4500 5800
+	1    0    0    -1
+$EndComp
+$Comp
+L Device:CP1 C8
+U 1 1 60E9992D
+P 4500 5650
+F 0 "C8" H 4600 5650 50  0000 L CNN
+F 1 "0.33uF" H 4550 5550 50  0000 L CNN
+F 2 "Capacitor_Tantalum_SMD:CP_EIA-3216-18_Kemet-A_Pad1.58x1.35mm_HandSolder" H 4500 5650 50  0001 C CNN
+F 3 "~" H 4500 5650 50  0001 C CNN
+	1    4500 5650
+	1    0    0    -1
+$EndComp
+Connection ~ 4500 5500
+$Comp
+L Device:CP1 C9
+U 1 1 60E9A065
+P 5150 5650
+F 0 "C9" H 5250 5650 50  0000 L CNN
+F 1 "0.1uF" H 5150 5550 50  0000 L CNN
+F 2 "Capacitor_Tantalum_SMD:CP_EIA-3216-18_Kemet-A_Pad1.58x1.35mm_HandSolder" H 5150 5650 50  0001 C CNN
+F 3 "~" H 5150 5650 50  0001 C CNN
+	1    5150 5650
 	1    0    0    -1
 $EndComp
 Wire Wire Line
-	4650 7150 4750 7150
-Connection ~ 4750 7150
-Wire Wire Line
-	4750 7150 5000 7150
-Wire Wire Line
-	4650 6350 4750 6350
-Connection ~ 4750 6350
-Wire Wire Line
-	4750 6350 5000 6350
+	5150 5500 5200 5500
+Connection ~ 5150 5500
 $Comp
-L Regulator_Linear:MC79M05_TO252 U9
-U 1 1 6216B584
-P 4850 5600
-F 0 "U9" H 4850 5451 50  0000 C CNN
-F 1 "MC79M05_TO252" H 4850 5360 50  0000 C CNN
-F 2 "Package_TO_SOT_SMD:TO-252-2" H 4850 5400 50  0001 C CIN
-F 3 "http://www.onsemi.com/pub/Collateral/MC79M00-D.PDF" H 4850 5600 50  0001 C CNN
-	1    4850 5600
+L power:GND #PWR0156
+U 1 1 60EBAE84
+P 5150 5800
+F 0 "#PWR0156" H 5150 5550 50  0001 C CNN
+F 1 "GND" V 5155 5672 50  0000 R CNN
+F 2 "" H 5150 5800 50  0001 C CNN
+F 3 "" H 5150 5800 50  0001 C CNN
+	1    5150 5800
 	1    0    0    -1
 $EndComp

Commit message: first routes.
Parts:
- added D7: LED_CLIP, LED_SMD:LED_0805_2012Metric_Pad1.15x1.40mm_HandSolder, symbol Device:LED
- added R19: 2k, Resistor_SMD:R_0805_2012Metric_Pad1.20x1.40mm_HandSolder, symbol Device:R
Connections:
- net +3V3: now also J2.19 (Pin_19), R19.2; no longer J2.20 (Pin_20)
- net +5V: now also J2.18 (Pin_18); no longer J2.19 (Pin_19)
- net -5V: now also J2.17 (Pin_17); no longer J2.18 (Pin_18)
- net GND: now also J2.20 (Pin_20), D7.1 (K); no longer J2.1 (Pin_1)
- net I2S_MUTE: now also J2.12 (Pin_12); no longer J2.8 (Pin_8)
- net I2S_SCK: now also J2.15 (Pin_15); no longer J2.6 (Pin_6)
- net I2S_SDA: now also J2.13 (Pin_13); no longer J2.7 (Pin_7)
- net I2S_WS: now also J2.14 (Pin_14); no longer J2.9 (Pin_9)
- net MIDI_IN: now also J2.3 (Pin_3); no longer J2.4 (Pin_4)
- net MIDI_IN_INV: now also J2.4 (Pin_4); no longer J2.12 (Pin_12)
- net UART_RX: now also J2.1 (Pin_1); no longer J2.2 (Pin_2)
- net UART_TX: now also J2.2 (Pin_2); no longer J2.3 (Pin_3)
- net MIDI_OUT_INV: now reaches R10.1, U5.6
- net MIDI_OUT_INV: now also J2.6 (Pin_6)
- new net: D7.2 (A), R19.1
Other:
- moved on the sheet: FB1, FB2, FB5, FB6, J3, J4, R10, R3, R4, R9, U5A, U5B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
