File: extended/xfm2.sch (KiCad schematic (older format))
At the start: 59 parts, among them J1 Midi In, J2 Pin Breakout, J3 Midi Out, J4 Midi Thru, J5 Conn_Coaxial, J6 Jack-DC, J7 A-100_Bus_Connector, J8 AudioJack2, J9 AudioJack2, U1 H11L1, U2 CmodA7-35T, U3 24LC01, U4 UDA1334A, U5 74HC14, U6 LM1117-5.0, U7 LM1117-3.3, U8 MCP6004, U9 L79L05_SO8

Commit message: fitted the 6.35mm audio jack which was too small. Added gerbers. ERC seems fine.
Parts:
- D7: value LED_CLIP -> LED_POWER
- J8, J9: footprint Connector_Audio:Jack_6.35mm_Neutrik_NRJ6HM-1_Horizontal -> xfm2:Jack_6.35mm_Neutrik_NMJ6HFD2_Horizontal-ST-only
Connections:
- net +5V: now also C2.1, U7.3 (VI)
- net GND: now also J8.S, J9.S; no longer J8.T, J9.T
- net at C3.1, D6.1 (K), U6.3 (VI): no longer C2.1, U7.3 (VI)
- net at R11.2: now also J8.T; no longer J8.S
- net at R12.2: now also J9.T; no longer J9.S
- no-connect marks 64 -> 66
Other:
- moved on the sheet: J8, J9
Changed lines of the file:
@@
 Sheet 1 1
 Title "xfm2/xva1 extended pcb"
-Date "2021-05-13"
+Date "2021-06-27"
 Rev "1.1"
 Comp ""
@@
 	1    0    0    -1
 $EndComp
-Wire Wire Line
-	3600 6350 3600 7150
-Connection ~ 3600 6350
 Text Notes 2750 5100 0    79   ~ 0
 Eurorack\nA-100
@@
 	1    0    0    -1
 $EndComp
-Wire Wire Line
-	3600 6350 3700 6350
 Wire Wire Line
 	3300 6550 3300 6700
@@
 U 1 1 610872B2
 P 4350 7150
-F 0 "U7" H 4150 7300 50  0000 C CNN
-F 1 "LM1117-3.3" H 4500 7300 50  0000 C CNN
+F 0 "U7" H 4450 6900 50  0000 C CNN
+F 1 "LM1117-3.3" H 4350 7300 50  0000 C CNN
 F 2 "Package_TO_SOT_SMD:SOT-223-3_TabPin2" H 4350 7150 50  0001 C CNN
 F 3 "http://www.ti.com/lit/ds/symlink/lm1117.pdf" H 4350 7150 50  0001 C CNN
@@
 	1    0    0    -1
 $EndComp
-Wire Wire Line
-	3750 7150 4050 7150
-Wire Wire Line
-	3600 7150 3750 7150
 Connection ~ 3750 7150
 $Comp
@@
 L Connector:AudioJack2 J8
 U 1 1 61995198
-P 1500 2450
-F 0 "J8" H 1532 2775 50  0000 C CNN
-F 1 "AudioJack2" H 1532 2684 50  0000 C CNN
-F 2 "Connector_Audio:Jack_6.35mm_Neutrik_NRJ6HM-1_Horizontal" H 1500 2450 50  0001 C CNN
-F 3 "~" H 1500 2450 50  0001 C CNN
-	1    1500 2450
+P 1300 2350
+F 0 "J8" H 1332 2675 50  0000 C CNN
+F 1 "AudioJack2" H 1332 2584 50  0000 C CNN
+F 2 "xfm2:Jack_6.35mm_Neutrik_NMJ6HFD2_Horizontal-ST-only" H 1300 2350 50  0001 C CNN
+F 3 "~" H 1300 2350 50  0001 C CNN
+	1    1300 2350
 	1    0    0    -1
 $EndComp
@@
 $EndComp
 Wire Wire Line
-	1700 2350 1750 2350
+	1500 2350 1750 2350
 $Comp
 L Device:R R11
@@
 L power:GND #PWR0150
 U 1 1 61B56DAD
-P 1700 2450
-F 0 "#PWR0150" H 1700 2200 50  0001 C CNN
-F 1 "GND" V 1705 2322 50  0000 R CNN
-F 2 "" H 1700 2450 50  0001 C CNN
-F 3 "" H 1700 2450 50  0001 C CNN
-	1    1700 2450
+P 1750 2000
+F 0 "#PWR0150" H 1750 1750 50  0001 C CNN
+F 1 "GND" V 1755 1872 50  0000 R CNN
+F 2 "" H 1750 2000 50  0001 C CNN
+F 3 "" H 1750 2000 50  0001 C CNN
+	1    1750 2000
 	1    0    0    -1
 $EndComp
@@
 L Connector:AudioJack2 J9
 U 1 1 61C477C6
-P 1500 3700
-F 0 "J9" H 1532 4025 50  0000 C CNN
-F 1 "AudioJack2" H 1532 3934 50  0000 C CNN
-F 2 "Connector_Audio:Jack_6.35mm_Neutrik_NRJ6HM-1_Horizontal" H 1500 3700 50  0001 C CNN
-F 3 "~" H 1500 3700 50  0001 C CNN
-	1    1500 3700
+P 1250 3600
+F 0 "J9" H 1282 3925 50  0000 C CNN
+F 1 "AudioJack2" H 1282 3834 50  0000 C CNN
+F 2 "xfm2:Jack_6.35mm_Neutrik_NMJ6HFD2_Horizontal-ST-only" H 1250 3600 50  0001 C CNN
+F 3 "~" H 1250 3600 50  0001 C CNN
+	1    1250 3600
 	1    0    0    -1
 $EndComp
@@
 	1    1900 3600
 	0    1    1    0
-$EndComp
-$Comp
-L power:GND #PWR0151
-U 1 1 61C483A4
-P 1700 3700
-F 0 "#PWR0151" H 1700 3450 50  0001 C CNN
-F 1 "GND" V 1705 3572 50  0000 R CNN
-F 2 "" H 1700 3700 50  0001 C CNN
-F 3 "" H 1700 3700 50  0001 C CNN
-	1    1700 3700
-	1    0    0    -1
 $EndComp
 $Comp
@@
 $EndComp
 Wire Wire Line
-	1700 3600 1750 3600
+	1450 3600 1750 3600
 Wire Wire Line
 	2050 3600 2100 3600
@@
 P 9300 6250
 F 0 "D7" H 9293 5995 50  0000 C CNN
-F 1 "LED_CLIP" H 9293 6086 50  0000 C CNN
+F 1 "LED_POWER" H 9293 6086 50  0000 C CNN
 F 2 "LED_SMD:LED_0805_2012Metric_Pad1.15x1.40mm_HandSolder" H 9300 6250 50  0001 C CNN
 F 3 "~" H 9300 6250 50  0001 C CNN
@@
 NoConn ~ 1150 6400
 NoConn ~ 6750 2650
+NoConn ~ 6350 400
+NoConn ~ 5050 5400
+Wire Wire Line
+	3750 7150 4050 7150
+Wire Wire Line
+	3600 6350 3700 6350
+Wire Wire Line
+	3600 7150 3750 7150
+$Comp
+L power:+5V #PWR0159
+U 1 1 60F43BCA
+P 3600 7150
+F 0 "#PWR0159" H 3600 7000 50  0001 C CNN
+F 1 "+5V" V 3615 7278 50  0000 L CNN
+F 2 "" H 3600 7150 50  0001 C CNN
+F 3 "" H 3600 7150 50  0001 C CNN
+	1    3600 7150
+	0    -1   -1   0
+$EndComp
+Wire Wire Line
+	1500 2250 1600 2250
+Wire Wire Line
+	1600 2250 1600 1950
+Wire Wire Line
+	1600 1950 1750 1950
+Wire Wire Line
+	1750 1950 1750 2000
+Wire Wire Line
+	1450 3500 1600 3500
+Wire Wire Line
+	1600 3500 1600 3200
+Wire Wire Line
+	1600 3200 1750 3200
+Wire Wire Line
+	1750 3200 1750 3250
+$Comp
+L power:GND #PWR0151
+U 1 1 61C483A4
+P 1750 3250
+F 0 "#PWR0151" H 1750 3000 50  0001 C CNN
+F 1 "GND" V 1755 3122 50  0000 R CNN
+F 2 "" H 1750 3250 50  0001 C CNN
+F 3 "" H 1750 3250 50  0001 C CNN
+	1    1750 3250
+	1    0    0    -1
+$EndComp
 $EndSCHEMATC

Commit message: updates for the extended xfm2 board: replacement of opamp components, logic level converter 5v<->3.3v and pull ups for uart.
Parts:
- added C10, C16: 47uF, Capacitor_SMD:CP_Elec_6.3x5.4, symbol Device:CP1
- added C11, C17, C18: 100nF, Capacitor_SMD:C_0805_2012Metric_Pad1.18x1.45mm_HandSolder, symbol Device:C
- added C12, C13: 100pF, Capacitor_SMD:C_0805_2012Metric_Pad1.18x1.45mm_HandSolder, symbol Device:C
- added C14, C15: 0.1uF, Capacitor_SMD:C_0805_2012Metric_Pad1.18x1.45mm_HandSolder, symbol Device:C
- added D8: 1N4007, Diode_SMD:D_MELF_Handsoldering, symbol Device:D
- added IC1, IC2: 74LVC1G07QSE-7, samacsys:SOT65P210X110-5N, symbol samacsys:74LVC1G07QSE-7
- added R20, R21, R22, R23: 10k, Resistor_SMD:R_0805_2012Metric_Pad1.20x1.40mm_HandSolder, symbol Device:R
- C8, C9: footprint Capacitor_Tantalum_SMD:CP_EIA-3216-18_Kemet-A_Pad1.58x1.35mm_HandSolder -> Capacitor_SMD:C_0805_2012Metric_Pad1.18x1.45mm_HandSolder; symbol Device:CP1 -> Device:C
- D1: value D -> 1N4148
- U3: value 24LC01 -> 24LC10
Connections:
- net +12V: no longer J7.10 (+12V), J7.9 (+12V)
- net +3V3: now also U8.10 (+), U8.12 (+), C10.1, C11.1, R20.1, R23.1
- net +5V: now also C17.1, C18.1, IC1.5 (VCC), IC2.5 (VCC), R21.2, R22.1; no longer J7.11 (+5V), J7.12 (+5V)
- net -12V: now also D8.1 (K); no longer C8.1, U9.2 (IN), U9.3 (IN), U9.6 (IN), U9.7 (IN)
- net -5V: now also C14.2, C15.2, C16.2
- net CV0_3.3V: now also C13.2
- net CV1_3.3V: now also C12.2
- net GND: now also U8.13 (-), U8.9 (-), C10.2, C11.2, C12.1, C13.1, C14.1, C15.1, C16.1, C17.2, C18.2, IC1.3 (GND), IC2.3 (GND)
- net UART_TX_5V: now reaches J2.7 (Pin_7)
- net UART_TX_5V: now also IC2.4 (Y), R21.1
- net UART_RX_5V: now reaches J2.8 (Pin_8)
- net UART_RX_5V: now also IC1.2 (A), R22.2
- net 5V-In: now reaches D6.2 (A), J6.1
- net 5V-In: now also J7.11 (+5V), J7.12 (+5V)
- net UART_RX renamed UART_TX_3.3V
- net UART_TX_3.3V: now also IC2.2 (A), R23.2
- net UART_TX renamed UART_RX_3.3V
- net UART_RX_3.3V: now also IC1.4 (Y), R20.2
- new net: C8.1, D8.2 (A), U9.2 (IN), U9.3 (IN), U9.6 (IN), U9.7 (IN)
- no-connect marks 66 -> 62
Other:
- note added: "External Connections"
- note added: "External RX 5V ->FPGA RX 3.3V"
- note added: "FPGA TX 3.3V -> External TX 5V"
- note added: "UART Voltage translation"
- moved on the sheet: C1, C2, C3, C4, C5, C6, C7, D2, D3, D4, D5, D6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
