File: extended/xfm2.sch (KiCad schematic (older format))
At the start: 75 parts, among them IC1 74LVC1G07QSE-7, IC2 74LVC1G07QSE-7, J1 Midi In, J2 Pin Breakout, J3 Midi Out, J4 Midi Thru, J5 Conn_Coaxial, J6 Jack-DC, J7 A-100_Bus_Connector, J8 AudioJack2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

Commit message: xfm2/xva pcb version 1.3 (untested, don't use yet).
Parts:
- removed C10, C16: 47uF, Capacitor_SMD:CP_Elec_6.3x5.4, symbol Device:CP1
- removed D6, D8: 1N4007, Diode_SMD:D_MELF_Handsoldering, symbol Device:D
- added C10: 1uF, Capacitor_SMD:C_0805_2012Metric_Pad1.18x1.45mm_HandSolder, symbol Device:C
- added C16: 0.1uF, Capacitor_SMD:C_0805_2012Metric_Pad1.18x1.45mm_HandSolder, symbol Device:C
- added C19: 10nF, Capacitor_SMD:C_0805_2012Metric_Pad1.18x1.45mm_HandSolder, symbol Device:C
- added D6, D8, D9: 1N5819/SS14, Diode_SMD:D_SMA-SMB_Universal_Handsoldering, symbol Device:D_Schottky
- added J10: 10137062-00021LF, samacsys:CONN_10137062-00021LF, symbol samacsys:10137062-00021LF
- added R24, R25: 5.1k, Resistor_SMD:R_0805_2012Metric_Pad1.20x1.40mm_HandSolder, symbol Device:R
- added U10: CY7C65213-28PVXI, Package_SO:SSOP-28_5.3x10.2mm_P0.65mm, symbol Interface_USB:CY7C65213-28PVXI
Connections:
- net +12V: now also J7.10 (+12V), J7.9 (+12V), D6.2 (A)
- net -12V: now also D8.1 (K)
- net -5V: no longer J2.17 (Pin_17)
- net GND: now also C10.2, C16.2, C19.2, J10.A1 (GND_1), J10.A12 (GND_2), J10.B1 (GND_3), J10.B12 (GND_4), R24.1, R25.1, U10.18 (GND), U10.21 (GND), U10.7 (GND)
- net UART_RX_5V: now also U10.1 (TXD)
- net UART_TX_5V: now also U10.5 (RXD)
- net at C8.1, U9.2 (IN), U9.3 (IN)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: now also D8.2 (A)
- net at C3.1, U6.3 (VI): now also D6.1 (K), D9.1 (K)
- removed net 5V-In: J6.1, J7.11 (+5V), J7.12 (+5V)
- net UART_RX_3.3V renamed UART_RX_3.3V_FPGA
- net UART_TX_3.3V renamed UART_TX_3.3V_FPGA
- new net: D9.2 (A), J6.1
- new net: C10.1, U10.17 (VCCD)
- new net: J10.A5 (CC1), R24.2
- new net: J10.B5 (CC2), R25.2
- new net D+: J10.A6 (DP1), U10.15 (USBDP)
- new net D-: J10.A7 (DN1), U10.16 (USBDM)
- new net VBUS: C16.1, C19.1, J10.A4 (VBUS_1), J10.A9 (VBUS_2), J10.B4 (VBUS_3), J10.B9 (VBUS_4), U10.20 (VCC), U10.4 (VCCIO)
- no-connect marks 62 -> 93
Other:
- note added: "USB to UART Bridge"
- moved on the sheet: C18, C2, C3, C4, C5, C8, IC2, J6, R21, R23, U6, U7

Commit message: Next bugfix version 1.33.
Parts:
- removed J10: 10137062-00021LF, samacsys:CONN_10137062-00021LF, symbol samacsys:10137062-00021LF
- added J10: USB4105-GF-A, GCT_USB4105-GF-A, symbol usb3-2:USB4105-GF-A
- C14, C15, C9: value 0.1uF -> 100nF
- C8: value 0.33uF -> 330nF
- IC1, IC2: footprint samacsys:SOT65P210X110-5N -> Package_TO_SOT_SMD:SOT-353_SC-70-5_Handsoldering; LCSC (none) -> C507244
- U1: LCSC (none) -> C20082
- U10: LCSC (none) -> C134181
- U6: LCSC (none) -> C23984
- U7: LCSC (none) -> C9662
- U8: LCSC (none) -> C7378
Connections:
- net D+: now also J10.A6 (DP1), J10.B6 (DP2)
- net D-: now also J10.A7 (DN1), J10.B7 (DN2)
- net UART_RX_5V: now also IC2.4 (Y), R21.1, U10.5 (RXD); no longer IC1.2 (A), R22.2, U10.1 (TXD)
- net UART_TX_5V: now also IC1.2 (A), R22.2, U10.1 (TXD); no longer IC2.4 (Y), R21.1, U10.5 (RXD)
- net VBUS: now also J10.B4_A9 (VBUS)
- net at R24.2: now also J10.B5 (CC2)
- net at R25.2: now also J10.A5 (CC1)
- no-connect marks 93 -> 82
Other:
- note added: "FPGA TX 3.3V -> UART RX 5V"
- note added: "UART TX 5V ->FPGA RX 3.3V"
- note removed: "External RX 5V ->FPGA RX 3.3V"
- note removed: "FPGA TX 3.3V -> External TX 5V"
- moved on the sheet: R24, R25

Commit message: missed a file...
Parts:
- J10: footprint GCT_USB4105-GF-A -> samacsys:GCT_USB4105-GF-A
Changed lines of the file:
@@
 F 0 "J10" H 4350 12717 50  0000 C CNN
 F 1 "USB4105-GF-A" H 4350 12626 50  0000 C CNN
-F 2 "GCT_USB4105-GF-A" H 4350 12050 50  0001 L BNN
+F 2 "samacsys:GCT_USB4105-GF-A" H 4350 12050 50  0001 L BNN
 F 3 "" H 4350 12050 50  0001 L BNN
 F 4 "A3" H 4350 12050 50  0001 L BNN "PARTREV"

Commit message: bugfix incl. gerber v1.34 for the extended board.
Parts:
- added C20: 10nF, Capacitor_SMD:C_0805_2012Metric_Pad1.18x1.45mm_HandSolder, symbol Device:C
- added C21: 0.1uF, Capacitor_SMD:C_0805_2012Metric_Pad1.18x1.45mm_HandSolder, symbol Device:C
- added D10: 1N5819/SS14, Diode_SMD:D_SMA-SMB_Universal_Handsoldering, symbol Device:D_Schottky
- added R26: 4.7k, Resistor_SMD:R_0805_2012Metric_Pad1.20x1.40mm_HandSolder, symbol Device:R
- added R27: 10k, Resistor_SMD:R_0805_2012Metric_Pad1.20x1.40mm_HandSolder, symbol Device:R
- IC1, IC2: footprint Package_TO_SOT_SMD:SOT-353_SC-70-5_Handsoldering -> greatscott:SOT25
Connections:
- net +5V: now also U10.4 (VCCIO), C20.2, C21.2, D10.1 (K); no longer C4.1, U6.2 (VO)
- net GND: now also J10.A1_B12 (GND), J10.B1_A12 (GND), C20.1, C21.1, R27.2
- net VBUS: now also J10.A4_B9 (VBUS), R26.1; no longer U10.4 (VCCIO)
- net at U10.19 (~RESET): now also R26.2, R27.1
- new net: C4.1, D10.2 (A), U6.2 (VO)
- no-connect marks 82 -> 83
Other:
- moved on the sheet: C16, C19, C2, C3, C4, C5, C8, C9, D2, D3, D4, D5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
