File: extended/xfm2.kicad_pcb (KiCad board)
At the start: 2 copper layers, 69.2 x 121.3 mm, 23 parts, among them J1 Midi In, J2 Pin Breakout, J3 Midi Out, J4 Midi Thru, J5 Conn_Coaxial, U1 4N36, U2 CmodA7-35T, U3 24LC01, U4 UDA1334A

Commit message: updated schematic
Parts:
- added FB1: Ferrite_Bead, Capacitor_SMD:C_0805_2012Metric_Pad1.18x1.45mm_HandSolder, F.Cu at (179.1, 119.4)
- added FB2: Ferrite_Bead, Capacitor_SMD:C_0805_2012Metric_Pad1.18x1.45mm_HandSolder, F.Cu at (179.6, 142.2)
- added FB3: Ferrite_Bead, Capacitor_SMD:C_0805_2012Metric_Pad1.18x1.45mm_HandSolder, F.Cu at (180.4, 90.4)
- added FB4: Ferrite_Bead, Capacitor_SMD:C_0805_2012Metric_Pad1.18x1.45mm_HandSolder, F.Cu at (178.8, 103.4)
- added FB5: Ferrite_Bead, Capacitor_SMD:C_0805_2012Metric_Pad1.18x1.45mm_HandSolder, F.Cu at (179.3, 126.2)
- added FB6: Ferrite_Bead, Capacitor_SMD:C_0805_2012Metric_Pad1.18x1.45mm_HandSolder, F.Cu at (179.6, 149.1)
- added R10: 10, Resistor_SMD:R_0805_2012Metric_Pad1.20x1.40mm_HandSolder, F.Cu at (179.3, 130.0)
- added R9: 10, Resistor_SMD:R_0805_2012Metric_Pad1.20x1.40mm_HandSolder, F.Cu at (179.6, 152.7)
- added U5: 74HC14, Package_SO:SO-14_3.9x8.65mm_P1.27mm, F.Cu at (170.4, 126.0)
- D1: footprint samacsys:SODFL1608X70N -> Diode_SMD:D_SOD-523
- D2: value LED_MIDI_1 -> LED_MIDI_IN
- D3: value LED_MIDI_2 -> LED_MIDI_OUT
- R5, R6, R7, R8: value 220 -> 2k
- U1: value 4N36 -> H11L1
- moved R2 5.86 mm to (167.6, 107.2)
- moved D1 3.48 mm to (178.8, 100.1)
- moved U1 3.21 mm to (171.2, 98.3), turned to 270 degrees
Connections:
- net /EEPROM_SCL renamed EEPROM_SCL
- net /EEPROM_SDA renamed EEPROM_SDA
- net /EEPROM_VCC renamed EEPROM_VCC
- D1 pad 2: /MIDI_TX_RETURN -> Net-(D1-Pad2)
- J1 pad 4: Net-(J1-Pad4) -> Net-(FB3-Pad1)
- J2 pad 10: I2S_SDA -> I2S_VCC
- J2 pad 11: MIDI_THRU -> SPDIF_OUT
- J2 pad 12: I2S_WS -> MIDI_IN_INV
- J2 pad 13: MIDI_IN -> Net-(J2-Pad13)
- J2 pad 14: I2S_MUTE -> Net-(J2-Pad14)
- J2 pad 15: SPDIF_OUT -> Net-(J2-Pad15)
- J2 pad 16: I2S_VCC -> Net-(J2-Pad16)
- J2 pad 20: Net-(J2-Pad20) -> VCC
- J2 pad 3: LED_MIDI_1 -> UART_TX
- J2 pad 4: UART_TX -> MIDI_IN
- J2 pad 5: LED_MIDI_2 -> MIDI_OUT
- J2 pad 6: MIDI_OUT -> I2S_SCK
- J2 pad 7: LED_AUDIO -> I2S_SDA
- J2 pad 8: I2S_SCK -> I2S_MUTE
- J2 pad 9: LED_CLIP -> I2S_WS
- J3 pad 2: Net-(J3-Pad2) -> GND
- J3 pad 4: Net-(J3-Pad4) -> Net-(FB1-Pad1)
- J3 pad 5: GND -> Net-(FB5-Pad2)
- J4 pad 2: Net-(J4-Pad2) -> GND
- J4 pad 4: Net-(J4-Pad4) -> Net-(FB6-Pad2)
- J4 pad 5: GND -> Net-(FB2-Pad1)
- R1 pad 1: Net-(J1-Pad4) -> Net-(FB3-Pad2)
- R2 pad 2: MIDI_IN_RETURN -> MIDI_IN
- R3 pad 1: Net-(J4-Pad4) -> I2S_VCC
- R3 pad 2: MIDI_THRU -> Net-(FB6-Pad1)
- R4 pad 1: Net-(J3-Pad4) -> Net-(FB1-Pad2)
- R4 pad 2: MIDI_OUT -> I2S_VCC
- R5 pad 2: LED_MIDI_1 -> MIDI_IN_INV
- R6 pad 2: LED_MIDI_2 -> MIDI_OUT
- U1 pad 2: /MIDI_TX_RETURN -> Net-(D1-Pad2)
- U1 pad 5: MIDI_IN_RETURN -> GND
- U1 pad 6: Net-(U1-Pad6) -> I2S_VCC
- U2 pad 37: LED_MIDI_1 -> Net-(U2-Pad37)
- U2 pad 38: LED_MIDI_2 -> Net-(U2-Pad38)
- U2 pad 41: MIDI_THRU -> Net-(U2-Pad41)
- U2 pad 42: MIDI_IN_RETURN -> MIDI_IN
- U2 pad 43: MIDI_IN -> Net-(U2-Pad43)
Routing:
- net MIDI_THRU: track 146.9 -> 0.00 mm, vias 1 -> 0
- net MIDI_OUT: track 146.3 -> 0.00 mm
- net LED_MIDI_1: track 125.5 -> 0.00 mm
- net LED_MIDI_2: track 123.6 -> 0.00 mm
- net LED_AUDIO: track 122.3 -> 0.00 mm
- net LED_CLIP: track 121.8 -> 0.00 mm
- net I2S_WS: track 115.2 -> 0.00 mm
- net I2S_SDA: track 111.7 -> 0.00 mm
- net I2S_SCK: track 109.1 -> 0.00 mm
- net I2S_MUTE: track 99.9 -> 0.00 mm
- net SPDIF_OUT: track 98.3 -> 0.00 mm, vias 1 -> 0
- net I2S_VCC: track 93.1 -> 0.00 mm
- net MIDI_IN: track 82.6 -> 0.00 mm, vias 2 -> 0
- net EEPROM_VCC: track 55.7 -> 0.00 mm, vias 2 -> 0
- net MIDI_IN_RETURN: track 39.6 -> 0.00 mm, vias 1 -> 0
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- removed copper zone on B.Cu, net GND
- removed copper zone on F.Cu, net GND
Other:
- board text added: "CV INPUT 0"
- board text added: "CV INPUT 1"
- board text added: "EEPROM GND"
- board text added: "EEPROM SCL"
- board text added: "EEPROM VCC"
- board text added: "EEPROM_SDA"
- board text added: "GND"
- board text added: "I2S MUTE"
- board text added: "I2S SCK"
- board text added: "I2S SDA"
- board text added: "I2S VCC"
- board text added: "I2S WS"
- board text added: "LED AUDIO"
- board text added: "LED CLIP"
- board text added: "LED MIDI 2"
- board text added: "LED MIDI INPUT"
- board text added: "MIDI IN"
- board text added: "MIDI IN RETURN"
- board text added: "MIDI OUT"
- board text added: "MIDI THRU"
- board text added: "Midi Input"
- board text added: "SPDIF OUT"
- board text added: "UART RX"
- board text added: "UART TX"
- board text added: "VCC"
- board text added: "xfm2/xva1 extended board v1.1"
- board text removed: "Midi 1"
- board text removed: "xfm2/xva1 extended board v1.0"

Commit message: initial extended pcb 1.1 placement
Parts:
- added C2: 10uF, Capacitor_SMD:C_0805_2012Metric_Pad1.18x1.45mm_HandSolder, F.Cu at (111.5, 186.4)
- added C3: 10uF, Capacitor_SMD:C_0805_2012Metric_Pad1.18x1.45mm_HandSolder, F.Cu at (111.5, 177.0)
- added C4: 100uF, Capacitor_SMD:CP_Elec_6.3x5.7, F.Cu at (131.8, 179.1)
- added C5: 100uF, Capacitor_SMD:CP_Elec_6.3x5.7, F.Cu at (131.6, 189.5)
- added C6: 330p-560p, Capacitor_SMD:C_0805_2012Metric_Pad1.18x1.45mm_HandSolder, F.Cu at (123.2, 56.9)
- added C7: 330p-560p, Capacitor_SMD:C_0805_2012Metric_Pad1.18x1.45mm_HandSolder, F.Cu at (122.7, 42.4)
- added D6: 1N4007, Diode_SMD:D_MELF_Handsoldering, F.Cu at (109.2, 181.4)
- added J6: Jack-DC, Connector_BarrelJack:BarrelJack_Wuerth_6941xx301002, F.Cu at (99.8, 181.4)
- added J7: A-100_Bus_Connector, Connector_PinHeader_2.54mm:PinHeader_2x08_P2.54mm_Vertical, F.Cu at (153.9, 183.9)
- added J8: AudioJack2, Connector_Audio:Jack_6.35mm_Neutrik_NRJ6HM-1_Horizontal, F.Cu at (103.9, 56.9)
- added J9: AudioJack2, Connector_Audio:Jack_6.35mm_Neutrik_NRJ6HM-1_Horizontal, F.Cu at (103.9, 37.6)
- added R11: 100k, Resistor_SMD:R_0805_2012Metric_Pad1.20x1.40mm_HandSolder, F.Cu at (117.3, 56.9)
- added R12: 100k, Resistor_SMD:R_0805_2012Metric_Pad1.20x1.40mm_HandSolder, F.Cu at (116.8, 37.6)
- added R13: 100k, Resistor_SMD:R_0805_2012Metric_Pad1.20x1.40mm_HandSolder, F.Cu at (117.3, 52.1)
- added R14: 100k, Resistor_SMD:R_0805_2012Metric_Pad1.20x1.40mm_HandSolder, F.Cu at (116.8, 42.4)
- added R15: 33k, Resistor_SMD:R_0805_2012Metric_Pad1.20x1.40mm_HandSolder, F.Cu at (123.2, 52.1)
- added R16: 33k, Resistor_SMD:R_0805_2012Metric_Pad1.20x1.40mm_HandSolder, F.Cu at (122.7, 37.6)
- added R17: 100, Resistor_SMD:R_0805_2012Metric_Pad1.20x1.40mm_HandSolder, F.Cu at (127.8, 56.9)
- added R18: 100, Resistor_SMD:R_0805_2012Metric_Pad1.20x1.40mm_HandSolder, F.Cu at (127.8, 42.4)
- added REF**: , MountingHole:MountingHole_2.7mm_M2.5, F.Cu at (89.7, 19.6)
- added REF**: , MountingHole:MountingHole_2.7mm_M2.5, F.Cu at (153.2, 19.6)
- added REF**: , MountingHole:MountingHole_2.7mm_M2.5, F.Cu at (153.2, 190.5)
- added REF**: , MountingHole:MountingHole_2.7mm_M2.5, F.Cu at (89.4, 190.5)
- added U6: LM1117-5.0, Package_TO_SOT_SMD:SOT-223-3_TabPin2, F.Cu at (120.4, 179.1)
- added U7: LM1117-3.3, Package_TO_SOT_SMD:SOT-223-3_TabPin2, F.Cu at (120.4, 189.5)
- added U8: MCP6004, Package_SO:SO-14_5.3x10.2mm_P1.27mm, F.Cu at (121.9, 30.7)
- added U9: MC79M05_TO252, Package_TO_SOT_SMD:TO-252-2, F.Cu at (129.5, 166.1)
- moved C1 169.9 mm to (92.5, 173.0), turned to 0 degrees
- moved J5 157.6 mm to (91.4, 165.0), turned to 0 degrees
- moved D2 138.1 mm to (128.7, 18.2), turned to 180 degrees
- moved D3 136.1 mm to (134.4, 18.2), turned to 180 degrees
- moved D4 135.0 mm to (140.1, 18.2), turned to 180 degrees
- moved D5 135.0 mm to (145.8, 18.2), turned to 180 degrees
- moved R5 128.5 mm to (127.8, 23.2), turned to 270 degrees
- moved R6 126.2 mm to (133.5, 23.2), turned to 270 degrees
- moved R7 125.0 mm to (139.2, 23.2), turned to 270 degrees
- moved R8 124.8 mm to (144.9, 23.2), turned to 270 degrees
- moved J4 122.2 mm to (95.8, 71.0), turned to 270 degrees
- moved R9 112.9 mm to (111.0, 63.0), turned to 180 degrees
- moved FB2 102.5 mm to (111.0, 66.0), turned to 0 degrees
- moved J3 101.7 mm to (95.8, 93.9), turned to 270 degrees
- moved FB6 100.1 mm to (111.3, 75.9), turned to 180 degrees
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Connections:
- J2 pad 10: I2S_VCC -> Net-(J2-Pad10)
- J2 pad 18: Net-(J2-Pad18) -> -5V
- J2 pad 19: Net-(J2-Pad19) -> +5V
- J2 pad 20: VCC -> +3V3
- R2 pad 1: EEPROM_VCC -> +3V3
- R3 pad 1: I2S_VCC -> +3V3
- R4 pad 2: I2S_VCC -> +3V3
- U1 pad 6: I2S_VCC -> +3V3
- U2 pad 15: Net-(U2-Pad15) -> CV0_3.3V
- U2 pad 16: Net-(U2-Pad16) -> CV1_3.3V
- U2 pad 24: VCC -> +5V
- U2 pad 36: I2S_VCC -> Net-(U2-Pad36)
- U2 pad 45: EEPROM_VCC -> Net-(U2-Pad45)
- U3 pad 3: EEPROM_VCC -> +3V3
- U3 pad 8: EEPROM_VCC -> +3V3
- U4 pad 1: I2S_VCC -> +3V3
- U4 pad 11: I2S_VCC -> +3V3
- U4 pad 13: I2S_VCC -> +3V3
- U5 pad 14: I2S_VCC -> +3V3
Other:
- board size 69.2 x 121.3 mm -> 70.6 x 178.1 mm
- board text added: "-5V"
- board text added: "24LC01"
- board text added: "3.3V"
- board text added: "5V"
- board text added: "74HC14"
- board text added: "A100 Bus Connector"
- board text added: "Analog Out"
- board text added: "CV IN0"
- board text added: "CV IN1"
- board text added: "CV0"
- board text added: "CV1"
- board text added: "DC 9-13V"
- board text added: "H11L1"
- board text added: "MCP6004"
- board text added: "Midi In"
- board text added: "Midi Out"
- board text added: "Midi Thru"
- board text added: "Pin Breakout"
- board text added: "Red Stripe"
- board text added: "SPDIF Out"
- board text removed: "Audio Out"
- board text removed: "CV INPUT 0"
- board text removed: "CV INPUT 1"
- board text removed: "EEPROM GND"
- board text removed: "EEPROM VCC"
- board text removed: "I2S VCC"
- board text removed: "LED MIDI 2"
- board text removed: "LED MIDI INPUT"
- board text removed: "MIDI IN RETURN"
- board text removed: "MIDI THRU"
- board text removed: "Midi 2"
- board text removed: "Midi Input"
- board text removed: "VCC"

Commit message: fixes
Parts:
- D1: footprint Diode_SMD:D_SOD-523 -> Diode_SMD:D_SOD-323_HandSoldering
Changed lines of the file:
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@@
-    )
-  )
-  (module Diode_SMD:D_SOD-523 (layer F.Cu)
-    (at 110.998 114.9985 180)
-    (descr "http://www.diodes.com/datasheets/ap02001.pdf p.144")
-    (tags "Diode SOD523")
-    (attr smd)
-    (fp_text reference D1 (at -0.762 -1.3335) (layer F.SilkS)
-      (effects (font (size 1 1) (thickness 0.15)))
-    )
-    (fp_text value D (at 0 1.4) (layer F.Fab)
-      (effects (font (size 1 1) (thickness 0.15)))
-    )
-    (fp_line (start 0.7 0.6) (end -1.15 0.6) (layer F.SilkS) (width 0.12))
-    (fp_line (start 0.7 -0.6) (end -1.15 -0.6) (layer F.SilkS) (width 0.12))
-    (fp_line (start 0.65 0.45) (end -0.65 0.45) (layer F.Fab) (width 0.1))
-    (fp_line (start -0.65 0.45) (end -0.65 -0.45) (layer F.Fab) (width 0.1))
-    (fp_line (start -0.65 -0.45) (end 0.65 -0.45) (layer F.Fab) (width 0.1))
-    (fp_line (start 0.65 -0.45) (end 0.65 0.45) (layer F.Fab) (width 0.1))
-    (fp_line (start -0.2 0.2) (end -0.2 -0.2) (layer F.Fab) (width 0.1))
-    (fp_line (start -0.2 0) (end -0.35 0) (layer F.Fab) (width 0.1))
-    (fp_line (start -0.2 0) (end 0.1 0.2) (layer F.Fab) (width 0.1))
-    (fp_line (start 0.1 0.2) (end 0.1 -0.2) (layer F.Fab) (width 0.1))
-    (fp_line (start 0.1 -0.2) (end -0.2 0) (layer F.Fab) (width 0.1))
-    (fp_line (start 0.1 0) (end 0.25 0) (layer F.Fab) (width 0.1))
-    (fp_line (start 1.25 0.7) (end -1.25 0.7) (layer F.CrtYd) (width 0.05))
-    (fp_line (start -1.25 0.7) (end -1.25 -0.7) (layer F.CrtYd) (width 0.05))
-    (fp_line (start -1.25 -0.7) (end 1.25 -0.7) (layer F.CrtYd) (width 0.05))
-    (fp_line (start 1.25 -0.7) (end 1.25 0.7) (layer F.CrtYd) (width 0.05))
-    (fp_line (start -1.15 -0.6) (end -1.15 0.6) (layer F.SilkS) (width 0.12))
-    (fp_text user %R (at 0 -1.3) (layer F.Fab)
-      (effects (font (size 1 1) (thickness 0.15)))
-    )
-    (pad 2 smd rect (at 0.7 0) (size 0.6 0.7) (layers F.Cu F.Paste F.Mask)
-      (net 61 "Net-(D1-Pad2)"))
-    (pad 1 smd rect (at -0.7 0) (size 0.6 0.7) (layers F.Cu F.Paste F.Mask)
-      (net 3 /MIDI_TX))
-    (model ${KISYS3DMOD}/Diode_SMD.3dshapes/D_SOD-523.wrl
-      (at (xyz 0 0 0))
-      (scale (xyz 1 1 1))
-      (rotate (xyz 0 0 0))
     )
   )
@@
       (at (xyz 0 0 0))
       (scale (xyz 1 1 1))
+      (rotate (xyz 0 0 0))
+    )
+  )
+  (module Diode_SMD:D_SOD-323_HandSoldering (layer F.Cu)
+    (at 110.998 114.9985 180)
+    (descr SOD-323)
+    (tags SOD-323)
+    (attr smd)
+    (fp_text reference D1 (at 0 -1.85) (layer F.SilkS)
+      (effects (font (size 1 1) (thickness 0.15)))
+    )
+    (fp_text value D (at 0.1 1.9) (layer F.Fab)
+      (effects (font (size 1 1) (thickness 0.15)))
+    )
+    (fp_line (start -1.9 -0.85) (end -1.9 0.85) (layer F.SilkS) (width 0.12))
+    (fp_line (start 0.2 0) (end 0.45 0) (layer F.Fab) (width 0.1))
+    (fp_line (start 0.2 0.35) (end -0.3 0) (layer F.Fab) (width 0.1))
+    (fp_line (start 0.2 -0.35) (end 0.2 0.35) (layer F.Fab) (width 0.1))
+    (fp_line (start -0.3 0) (end 0.2 -0.35) (layer F.Fab) (width 0.1))
+    (fp_line (start -0.3 0) (end -0.5 0) (layer F.Fab) (width 0.1))
+    (fp_line (start -0.3 -0.35) (end -0.3 0.35) (layer F.Fab) (width 0.1))
+    (fp_line (start -0.9 0.7) (end -0.9 -0.7) (layer F.Fab) (width 0.1))
+    (fp_line (start 0.9 0.7) (end -0.9 0.7) (layer F.Fab) (width 0.1))
+    (fp_line (start 0.9 -0.7) (end 0.9 0.7) (layer F.Fab) (width 0.1))
+    (fp_line (start -0.9 -0.7) (end 0.9 -0.7) (layer F.Fab) (width 0.1))
+    (fp_line (start -2 -0.95) (end 2 -0.95) (layer F.CrtYd) (width 0.05))
+    (fp_line (start 2 -0.95) (end 2 0.95) (layer F.CrtYd) (width 0.05))
+    (fp_line (start -2 0.95) (end 2 0.95) (layer F.CrtYd) (width 0.05))
+    (fp_line (start -2 -0.95) (end -2 0.95) (layer F.CrtYd) (width 0.05))
+    (fp_line (start -1.9 0.85) (end 1.25 0.85) (layer F.SilkS) (width 0.12))
+    (fp_line (start -1.9 -0.85) (end 1.25 -0.85) (layer F.SilkS) (width 0.12))
+    (fp_text user %R (at 0 -1.85) (layer F.Fab)
+      (effects (font (size 1 1) (thickness 0.15)))
+    )
+    (pad 1 smd rect (at -1.25 0 180) (size 1 1) (layers F.Cu F.Paste F.Mask)
+      (net 3 /MIDI_TX))
+    (pad 2 smd rect (at 1.25 0 180) (size 1 1) (layers F.Cu F.Paste F.Mask)
+      (net 61 "Net-(D1-Pad2)"))
+    (model ${KISYS3DMOD}/Diode_SMD.3dshapes/D_SOD-323.wrl
+      (at (xyz 0 0 0))
+      (scale (xyz 1 1 1))

Commit message: power updates.
Parts:
- removed REF** (x4): , MountingHole:MountingHole_2.7mm_M2.5
- added C8: 0.33uF, Capacitor_Tantalum_SMD:CP_EIA-3216-18_Kemet-A_Pad1.58x1.35mm_HandSolder, F.Cu at (233.0, 100.6)
- added C9: 0.1uF, Capacitor_Tantalum_SMD:CP_EIA-3216-18_Kemet-A_Pad1.58x1.35mm_HandSolder, F.Cu at (222.1, 100.6)
- C4, C5: value 100uF -> 10uF; footprint Capacitor_SMD:CP_Elec_6.3x5.7 -> Capacitor_Tantalum_SMD:CP_EIA-3216-18_Kemet-A_Pad1.58x1.35mm_HandSolder
- U9: value MC79M05_TO252 -> L79L05_SO8; footprint Package_TO_SOT_SMD:TO-252-2 -> Package_SO:SOIC-8_3.9x4.9mm_P1.27mm
- moved C2 144.9 mm to (240.4, 120.3), turned to 270 degrees
- moved J6 136.4 mm to (230.1, 141.0), turned to 0 degrees
- moved U7 134.1 mm to (235.3, 120.4), turned to 90 degrees
- moved C1 131.6 mm to (221.7, 148.3), turned to 90 degrees
- moved D6 130.8 mm to (230.1, 131.6), turned to 270 degrees
- moved C3 127.1 mm to (225.2, 120.3), turned to 270 degrees
- moved J7 125.0 mm to (232.7, 86.9), turned to 270 degrees
- moved J5 123.3 mm to (213.7, 149.4), turned to 90 degrees
- moved C5 120.4 mm to (230.1, 120.3), turned to 270 degrees
- moved U9 117.8 mm to (227.5, 100.6)
- moved U6 115.7 mm to (220.1, 120.4), turned to 90 degrees
- moved D2 112.4 mm to (66.9, 112.1), turned to 270 degrees
- moved D3 111.0 mm to (66.9, 106.4), turned to 270 degrees
- moved D4 110.3 mm to (66.9, 100.7), turned to 270 degrees
- moved D5 110.1 mm to (66.9, 95.0), turned to 270 degrees
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Connections:
- U9 pad 1: GND -> -5V
- U9 pad 3: -5V -> -12V
Other:
- board size 70.6 x 178.1 mm -> 178.1 x 70.6 mm
- board text removed: "-5V"
- board text removed: "24LC01"
- board text removed: "3.3V"
- board text removed: "5V"
- board text removed: "74HC14"
- board text removed: "H11L1"
- board text removed: "MCP6004"
- board text removed: "UDA1334"

Commit message: first routes.
Parts:
- added D7: LED_CLIP, LED_SMD:LED_0805_2012Metric_Pad1.15x1.40mm_HandSolder, F.Cu at (66.9, 94.4)
- added R19: 2k, Resistor_SMD:R_0805_2012Metric_Pad1.20x1.40mm_HandSolder, F.Cu at (70.4, 94.4)
- added REF**: MountingHole_2.7mm_M2.5, MountingHole:MountingHole_2.7mm_M2.5, F.Cu at (239.5, 87.4)
- added REF**: MountingHole_2.7mm_M2.5, MountingHole:MountingHole_2.7mm_M2.5, F.Cu at (239.5, 151.4)
- added REF**: MountingHole_2.7mm_M2.5, MountingHole:MountingHole_2.7mm_M2.5, F.Cu at (68.1, 151.4)
- added REF**: MountingHole_2.7mm_M2.5, MountingHole:MountingHole_2.7mm_M2.5, F.Cu at (68.1, 87.4)
- moved R6 5.08 mm to (70.4, 111.4)
- moved R8 5.08 mm to (70.4, 100.0)
- moved D2 5.08 mm to (66.9, 117.1)
- moved D3 5.08 mm to (66.9, 111.5)
- moved D4 5.08 mm to (66.9, 105.8)
- moved D5 5.08 mm to (66.9, 100.1)
- moved R5 5.08 mm to (70.4, 117.1)
- moved R7 5.08 mm to (70.4, 105.7)
- moved C8 0.38 mm to (232.7, 100.6)
- moved C9 0.38 mm to (221.7, 100.6)
- moved U9 0.38 mm to (227.1, 100.6)
- moved C5 0.13 mm to (230.1, 120.4)
- moved R3 0.13 mm to (127.8, 129.5)
- turned D1 to 90 degrees
Connections:
- J2 pad 1: GND -> UART_RX
- J2 pad 12: MIDI_IN_INV -> I2S_MUTE
- J2 pad 13: Net-(J2-Pad13) -> I2S_SDA
- J2 pad 14: Net-(J2-Pad14) -> I2S_WS
- J2 pad 15: Net-(J2-Pad15) -> I2S_SCK
- J2 pad 17: Net-(J2-Pad17) -> -5V
- J2 pad 18: -5V -> +5V
- J2 pad 19: +5V -> +3V3
- J2 pad 2: UART_RX -> UART_TX
- J2 pad 20: +3V3 -> GND
- J2 pad 3: UART_TX -> MIDI_IN
- J2 pad 4: MIDI_IN -> MIDI_IN_INV
- J2 pad 6: I2S_SCK -> MIDI_OUT_INV
- J2 pad 7: I2S_SDA -> Net-(J2-Pad7)
- J2 pad 8: I2S_MUTE -> Net-(J2-Pad8)
- J2 pad 9: I2S_WS -> Net-(J2-Pad9)
- R10 pad 1: Net-(R10-Pad1) -> MIDI_OUT_INV
- U5 pad 6: Net-(R10-Pad1) -> MIDI_OUT_INV
Routing:
- net (no net): track 0.00 -> 48.3 mm
- net Net-(C2-Pad1): track 0.00 -> 41.8 mm
- net +3V3: track 0.00 -> 38.3 mm
- net +5V: track 0.00 -> 31.7 mm
- net -5V: track 0.00 -> 28.7 mm, vias 0 -> 1
- net -12V: track 0.00 -> 26.4 mm
- net Net-(C7-Pad2): track 0.00 -> 14.1 mm
- net Net-(D1-Pad2): track 0.00 -> 13.7 mm
- net /MIDI_TX: track 0.00 -> 13.0 mm
- net Net-(C7-Pad1): track 0.00 -> 11.1 mm
- net Net-(C6-Pad2): track 0.00 -> 10.4 mm
- net Net-(FB3-Pad1): track 0.00 -> 9.92 mm
- net Net-(FB2-Pad1): track 0.00 -> 8.98 mm
- net Net-(FB5-Pad2): track 0.00 -> 8.98 mm
- net Net-(FB1-Pad1): track 0.00 -> 8.98 mm
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Other:
- net class 12v added: clearance 0.2, trace_width 1.5, via_dia 2, via_drill 0.4
- net class power 3-5v added: clearance 0.2, trace_width 0.5, via_dia 0.8, via_drill 0.4
- board text added: "Power"
