File: ui-board/kicad/xfm2-ui-board/xfm2-ui-board.kicad_pcb (KiCad board)
At the start: 2 copper layers, 353.6 x 95.5 mm, 87 parts, among them IC1 BR24T1MF-3AME2 EEPROM (0x50/1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, J1 XFM2/XVA1 Extended Board Conn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, J2 AVR-ISP-6, J3 ERM24064, J4 USB4105-GF-A, SW1 Reset, SW10 F7, SW11 Edit_Compare, SW12 2, SW13 Down, SW14 8, SW15 Page Next, SW16 F2, SW17 F8, SW18 Copy, SW19 3, SW2 Shift, SW20 9, SW21 Bank / Select, SW22 Left, SW23 F3, SW24 Exit, SW25 Memory, SW26 0, SW27 4, SW28 Element, SW29 F4, SW3 F6, SW30 Right, SW31 EF Bypass, SW32 Sign, SW33 F5, SW34 5, SW35 -1/No, SW36 Operator, SW37 6, SW38 Enter, SW39 +1/Yes, SW4 Utility, SW40 Knob 1, SW41 Knob 5, SW42 Data Entry Rotary, SW43 Knob 2, SW44 Knob 6, SW45 Knob 3, SW46 Volume, SW47 Knob 4, SW48 Jump, SW49 Voice, SW5 1, SW50 Multi, SW6 7, SW7 Up, SW8 Page Previous, SW9 F1, U1 ATMEGA2560-16AU, U2 MCP23017_SO (0x20), U3 MCP23017_SO (0x21), U4 MCP23017_SO (0x22), U5 CY7C65213-28PVXI, Y1 Crystal 16MHz

Commit message: lots of ui board routing
Parts:
- added J5: SPI Pins, Connector_PinHeader_2.54mm:PinHeader_1x06_P2.54mm_Vertical, F.Cu at (113.0, 41.9)
- added R13: 4.7k, Resistor_SMD:R_0805_2012Metric_Pad1.20x1.40mm_HandSolder, F.Cu at (170.2, 87.4)
- added R14: 4.7k, Resistor_SMD:R_0805_2012Metric_Pad1.20x1.40mm_HandSolder, F.Cu at (170.2, 85.3)
- added U6: MCP23017_SO (0x24), Package_SO:SOIC-28W_7.5x17.9mm_P1.27mm, F.Cu at (158.5, 85.9)
- moved J2 126.7 mm to (122.2, 41.7), turned to 90 degrees
- moved C3 107.7 mm to (129.6, 51.7)
- moved C4 107.7 mm to (129.6, 53.7)
- moved U1 94.6 mm to (128.4, 64.9), turned to 270 degrees
- moved C1 88.6 mm to (116.7, 61.7), turned to 180 degrees
- moved Y1 88.6 mm to (116.7, 63.8)
- moved C2 88.5 mm to (116.7, 65.8), turned to 180 degrees
- moved RV2 74.7 mm to (45.7, 54.4)
- moved RV1 67.3 mm to (30.8, 54.4)
- moved IC1 59.9 mm to (110.5, 69.8)
- moved R7 26.7 mm to (28.3, 103.6), turned to 180 degrees
- moved R6 23.8 mm to (28.3, 105.7)
- moved R5 17.5 mm to (303.3, 113.8), turned to 180 degrees
- moved C7 16.9 mm to (20.2, 112.0), turned to 90 degrees
- moved C6 16.8 mm to (18.2, 112.0), turned to 270 degrees
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Connections:
- J1 pad 7: /UART_TX_5V -> /RX1_D45
- J1 pad 8: /UART_RX_5V -> /TX1_D46
- SW40 pad A1: /D32 -> /D37
- SW40 pad C1: /D33 -> /D36
- SW41 pad A1: /D40 -> /D39
- SW41 pad C1: /D41 -> /D29
- SW42 pad A: /D30 -> /D26
- SW42 pad B: /D31 -> /D25
- SW43 pad A1: /D34 -> /D35
- SW43 pad C1: /D35 -> /D34
- SW44 pad A1: /D26 -> /D28
- SW45 pad A1: /D36 -> /D33
- SW45 pad C1: /D37 -> /D32
- SW46 pad A1: /D28 -> /D41
- SW46 pad C1: /D29 -> /D40
- SW47 pad A1: /D38 -> /D31
- SW47 pad C1: /D39 -> /D30
- U2 pad 21: /Numpad_8 -> Net-(U2-Pad21)
- U2 pad 22: /Numpad_9 -> Net-(U2-Pad22)
- U2 pad 23: /Numpad_Sign -> Net-(U2-Pad23)
- U2 pad 24: /Numpad_Enter -> Net-(U2-Pad24)
- U2 pad 25: /DPad_Up -> /Numpad_9
- U2 pad 26: /DPad_Down -> /Numpad_6
- U2 pad 27: /DPad_Left -> /Numpad_3
- U2 pad 28: /DPad_Right -> /Numpad_Enter
- U2 pad 3: /Numpad_2 -> /Numpad_4
- U2 pad 4: /Numpad_3 -> /Numpad_7
- U2 pad 5: /Numpad_4 -> /Numpad_Sign
- U2 pad 6: /Numpad_5 -> /Numpad_2
- U2 pad 7: /Numpad_6 -> /Numpad_5
- U2 pad 8: /Numpad_7 -> /Numpad_8
- U3 pad 1: /DPad_No -> /DPad_Left
- U3 pad 2: /DPad_Yes -> /DPad_No
- U3 pad 21: /FK_F1 -> Net-(U3-Pad21)
- U3 pad 22: /FK_F2 -> Net-(U3-Pad22)
- U3 pad 23: /FK_F3 -> Net-(U3-Pad23)
- U3 pad 24: /FK_F4 -> Net-(U3-Pad24)
- U3 pad 25: /FK_F5 -> /DPad_Operator
- U3 pad 26: /FK_F6 -> /DPad_Jump
- U3 pad 27: /FK_F7 -> /DPad_Yes
- U3 pad 28: /FK_F8 -> /DPad_Right
- U3 pad 4: /DPad_Page_Next -> /DPad_Select
- U3 pad 5: /DPad_Select -> /DPad_Down
- U3 pad 6: /DPad_Element -> /DPad_Up
- U3 pad 7: /DPad_Operator -> /DPad_Page_Next
- U3 pad 8: /FK_Shift -> /DPad_Element
- U4 pad 1: /FK_Exit -> /MD_EF_Bypass
- U4 pad 2: /MD_Utility -> /MD_Edit
- U4 pad 21: /MD_Multi -> Net-(U4-Pad21)
- U4 pad 25: Net-(U4-Pad25) -> /MD_Utility
- U4 pad 26: Net-(U4-Pad26) -> /MD_Memory
- U4 pad 27: Net-(U4-Pad27) -> /MD_Multi
- U4 pad 28: Net-(U4-Pad28) -> /MD_Copy
- U4 pad 3: /MD_Edit -> /MD_Voice
- U4 pad 4: /MD_Copy -> Net-(U4-Pad4)
- U4 pad 5: /MD_Memory -> Net-(U4-Pad5)
- U4 pad 6: /MD_EF_Bypass -> Net-(U4-Pad6)
- U4 pad 7: /DPad_Jump -> Net-(U4-Pad7)
- U4 pad 8: /MD_Voice -> Net-(U4-Pad8)
Routing:
- net /D27: track 0.00 -> 132.7 mm, vias 0 -> 2
- net /D28: track 0.00 -> 124.0 mm, vias 0 -> 2
- net /D29: track 0.00 -> 112.0 mm, vias 0 -> 2
- net /D39: track 0.00 -> 102.8 mm, vias 0 -> 2
- net /D30: track 0.00 -> 97.4 mm, vias 0 -> 2
- net /FK_Exit: track 0.00 -> 92.3 mm, vias 0 -> 1
- net /D41: track 0.00 -> 91.7 mm, vias 0 -> 3
- net /D31: track 0.00 -> 88.6 mm, vias 0 -> 2
- net +5V: track 0.00 -> 85.2 mm, vias 0 -> 8
- net /D40: track 0.00 -> 82.7 mm, vias 0 -> 3
- net /D37: track 0.00 -> 80.0 mm, vias 0 -> 3
- net /FK_Shift: track 0.00 -> 77.4 mm, vias 0 -> 1
- net /D32: track 0.00 -> 76.8 mm, vias 0 -> 2
- net /FK_F8: track 0.00 -> 74.5 mm, vias 0 -> 1
- net /D36: track 0.00 -> 69.6 mm, vias 0 -> 3
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- added copper zone on B.Cu, net GND
- added copper zone on F.Cu, net GND
Other:
- board size 353.6 x 95.5 mm -> 354.3 x 96.5 mm
- board text added: "+5V"
- board text added: "GND"
- board text added: "MISO"
- board text added: "MOSI"
- board text added: "SCK"

Commit message: fully routed.
Parts:
- J5: value SPI Pins -> SPI
Routing:
- net +5V: track 85.2 -> 993.8 mm, vias 8 -> 33
- net /SDA_D20: track 60.4 -> 426.1 mm, vias 0 -> 8
- net /SCL_D21: track 67.4 -> 427.0 mm, vias 2 -> 12
- net /AVR_TX: track 0.00 -> 166.0 mm, vias 0 -> 4
- net /AVR_RX: track 0.00 -> 165.6 mm, vias 0 -> 4
- net /RX1_D45: track 0.00 -> 159.4 mm, vias 0 -> 4
- net /A0: track 0.00 -> 159.3 mm, vias 0 -> 2
- net /TX1_D46: track 0.00 -> 156.9 mm, vias 0 -> 4
- net /D26: track 0.00 -> 146.1 mm, vias 0 -> 2
- net /D25: track 0.00 -> 141.4 mm
- net /RESET: track 13.3 -> 151.1 mm, vias 0 -> 3
- net /D4: track 0.00 -> 96.9 mm, vias 0 -> 4
- net /D5: track 0.00 -> 94.2 mm, vias 0 -> 4
- net /RX2_D17: track 0.00 -> 93.8 mm, vias 0 -> 2
- net /D6: track 0.00 -> 73.6 mm, vias 0 -> 4
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
Commit message: small corrections + mounting holes.
Parts:
- added REF**: MountingHole_3.2mm_M3_DIN965_Pad_TopBottom, MountingHole:MountingHole_3.2mm_M3_DIN965_Pad_TopBottom, F.Cu at (11.2, 133.6)
- added REF**: MountingHole_3.2mm_M3_DIN965_Pad_TopBottom, MountingHole:MountingHole_3.2mm_M3_DIN965_Pad_TopBottom, F.Cu at (367.8, 37.3)
- added REF**: MountingHole_3.2mm_M3_DIN965_Pad_TopBottom, MountingHole:MountingHole_3.2mm_M3_DIN965_Pad_TopBottom, F.Cu at (367.8, 133.3)
- added REF**: MountingHole_3.2mm_M3_DIN965_Pad_TopBottom, MountingHole:MountingHole_3.2mm_M3_DIN965_Pad_TopBottom, F.Cu at (11.2, 37.3)
- moved C5 2.79 mm to (26.2, 79.8)
Routing:
- net +5V: track 993.8 -> 997.8 mm
Other:
- board size 354.3 x 96.5 mm -> 363.7 x 103.4 mm

Commit message: small changes + gerber for front panel dev board
Other:
- board text added: "XVA1/XFM2 Front Panel Dev Board 0.90"

Commit message: updated footprint for the crystal
Parts:
- J5: value SPI -> SPI Pins
- Y1: footprint Crystal:Crystal_SMD_2012-2Pin_2.0x1.2mm_HandSoldering -> Crystal:Crystal_SMD_3225-4Pin_3.2x2.5mm_HandSoldering
- moved Y1 9.03 mm to (107.7, 63.2), turned to 270 degrees
Routing:
- net Net-(C2-Pad1): track 5.49 -> 18.6 mm
- net Net-(C1-Pad1): track 6.07 -> 17.1 mm
- net GND: track 34.9 -> 36.7 mm, vias 17 -> 18
