File: ui-board/kicad/xfm2-ui-board/xfm2-ui-board.sch (KiCad schematic (older format))
At the start: 72 parts, among them IC1 BR24T1MF-3AME2 EEPROM (0x50/1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, J1 XFM2/XVA1 Extended Board Conn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, J2 AVR-ISP-6, J3 ERM24064, SW1 Arduino Reset Pusbutton, SW10 F7, SW11 Edit_Compare, SW12 2, SW13 Down, SW14 8, SW15 Page Next, SW16 F2, SW17 F8, SW18 Copy, SW19 3, SW2 Shift, SW20 9, SW21 Bank / Select, SW22 Left, SW23 F3, SW24 Exit, SW25 Memory, SW26 0, SW27 4, SW28 Element, SW29 F4, SW3 F6, SW30 Right, SW31 EF Bypass, SW32 Sign, SW33 F5, SW34 5, SW35 -1/No, SW36 Operator, SW37 6, SW38 Enter, SW39 +1/Yes, SW4 Utility, SW40 Knob 5, SW41 Knob 6, SW42 Data Entry Rotary, SW43 Knob 1, SW44 Knob 2, SW45 Knob 3, SW46 Knob 4, SW47 Volume, SW5 1, SW6 7, SW7 Up, SW8 Page Previous, SW9 F1, U1 ATMEGA2560-16AU, U2 MCP23017_SO (0x20), U3 MCP23017_SO (0x21), U4 MCP23017_SO (0x22), Y1 Crystal

Commit message: unwired ui develeopment board is mostly done.
Parts:
- removed SW40: Knob 5, symbol Device:Rotary_Encoder_Switch
- removed SW41: Knob 6, symbol Device:Rotary_Encoder_Switch
- removed SW43: Knob 1, symbol Device:Rotary_Encoder_Switch
- removed SW44: Knob 2, symbol Device:Rotary_Encoder_Switch
- removed SW45: Knob 3, symbol Device:Rotary_Encoder_Switch
- removed SW46: Knob 4, symbol Device:Rotary_Encoder_Switch
- removed SW47: Volume, symbol Device:Rotary_Encoder_Switch
- added C10: 1uF, Capacitor_SMD:C_0805_2012Metric_Pad1.18x1.45mm_HandSolder, symbol Device:C
- added C6, C8: 4.7uF, Capacitor_SMD:C_0805_2012Metric_Pad1.18x1.45mm_HandSolder, symbol Device:C
- added C7, C9: 0.1uF, Capacitor_SMD:C_0805_2012Metric_Pad1.18x1.45mm_HandSolder, symbol Device:C
- added D1: LED, LED_SMD:LED_0805_2012Metric_Pad1.15x1.40mm_HandSolder, symbol Device:LED
- added J4: USB4105-GF-A, samacsys:GCT_USB4105-GF-A, symbol USB4105:USB4105-GF-A
- added R10, R11: 5.1k, Resistor_SMD:R_0805_2012Metric_Pad1.20x1.40mm_HandSolder, symbol Device:R
- added R12: 2k, Resistor_SMD:R_0805_2012Metric_Pad1.20x1.40mm_HandSolder, symbol Device:R
- added R8: 4.7k, Resistor_SMD:R_0805_2012Metric_Pad1.20x1.40mm_HandSolder, symbol Device:R
- added R9: 10k, Resistor_SMD:R_0805_2012Metric_Pad1.20x1.40mm_HandSolder, symbol Device:R
- added SW40: Knob 1, samacsys:PEC164015FN0024, symbol PEC16-4015F:PEC16-4015F-N0024
- added SW41: Knob 5, samacsys:PEC164015FN0024, symbol PEC16-4015F:PEC16-4015F-N0024
- added SW43: Knob 2, samacsys:PEC164015FN0024, symbol PEC16-4015F:PEC16-4015F-N0024
- added SW44: Knob 6, samacsys:PEC164015FN0024, symbol PEC16-4015F:PEC16-4015F-N0024
- added SW45: Knob 3, samacsys:PEC164015FN0024, symbol PEC16-4015F:PEC16-4015F-N0024
- added SW46: Volume, samacsys:PEC164015FN0024, symbol PEC16-4015F:PEC16-4015F-N0024
- added SW47: Knob 4, samacsys:PEC164015FN0024, symbol PEC16-4015F:PEC16-4015F-N0024
- added SW48: Jump, Button_Switch_THT:SW_PUSH_6mm, symbol Switch:SW_Push
- added SW49: Voice, Button_Switch_THT:SW_PUSH_6mm, symbol Switch:SW_Push
- added SW50: Multi, Button_Switch_THT:SW_PUSH_6mm, symbol Switch:SW_Push
- C1, C2: value C -> 18-22pF
- C3: value C -> 10nF
- C4: value C -> 100nF
- C5: value CP -> 100uF
- J2: footprint (none) -> Connector_PinHeader_2.54mm:PinHeader_1x06_P2.54mm_Vertical
- J3: footprint (none) -> Connector_PinHeader_2.54mm:PinHeader_2x11_P2.54mm_Vertical
- R1: value R -> 10k; footprint (none) -> Resistor_SMD:R_0805_2012Metric_Pad1.20x1.40mm_HandSolder
- R2, R3, R4, R5, R6, R7: footprint (none) -> Resistor_SMD:R_0805_2012Metric_Pad1.20x1.40mm_HandSolder
- RV1, RV2: footprint (none) -> Potentiometer_THT:Potentiometer_ACP_CA9-V10_Vertical
- RV3: footprint (none) -> samacsys:RS30111A9012
- SW1, SW10, SW11, SW12, SW13, SW14, SW15, SW16, SW17, SW18, SW19, SW2, SW20, SW21, SW22, SW23, SW24, SW25, SW26, SW27, SW28, SW29, SW3, SW30, SW31, SW32, SW33, SW34, SW35, SW36, SW37, SW38, SW39, SW4, SW5, SW6, SW7, SW8, SW9: footprint (none) -> Button_Switch_THT:SW_PUSH_6mm
- SW42: footprint (none) -> Rotary_Encoder:RotaryEncoder_Alps_EC11E-Switch_Vertical_H20mm
- Y1: value Crystal -> Crystal 16MHz; footprint (none) -> Crystal:Crystal_SMD_2012-2Pin_2.0x1.2mm_HandSoldering
- gave numbers to parts that had none: 1
Connections:
- net RX0 is gone; now on net AVR_TX: U1.2 (PE0(RXD0/PCINT8))
- net TX0 is gone; now on net AVR_RX: U1.3 (PE1(TXD0))
- net +5V: now also U5.4 (VCCIO), C6.2, C7.1, R12.2
- net -5V: no longer J1.17 (Pin_17)
- net D26: now also SW44.A1 (CCW)
- net D27: now also SW44.C1 (CW)
- net D28: now also SW46.A1 (CCW)
- net D29: now also SW46.C1 (CW)
- net D30: now also SW42.A
- net D31: now also SW42.B
- net D32: now also SW40.A1 (CCW)
- net D33: now also SW40.C1 (CW)
- net D34: now also SW43.A1 (CCW)
- net D35: now also SW43.C1 (CW)
- net D36: now also SW45.A1 (CCW)
- net D37: now also SW45.C1 (CW)
- net D38: now also SW47.A1 (CCW)
- net D39: now also SW47.C1 (CW)
- net D40: now also SW41.A1 (CCW)
- net D41: now also SW41.C1 (CW)
- net GND: now also U5.18 (GND), U5.21 (GND), U5.7 (GND), C10.1, C6.1, C7.2, C8.2, C9.1, D1.1 (K), J4.A1_B12 (GND), J4.B1_A12 (GND), R10.2, R11.2, R9.2, SW40.B1 (WIPER), SW41.B1 (WIPER), SW43.B1 (WIPER), SW44.B1 (WIPER), SW45.B1 (WIPER), SW46.B1 (WIPER), SW47.B1 (WIPER), SW48.2, SW49.2, SW50.2
- net AVR_TX: now reaches U5.1 (TXD)
- net D+: now reaches U5.15 (USBDP)
- net D+: now also J4.A6 (DP1), J4.B6 (DP2)
- net D-: now reaches U5.16 (USBDM)
- net D-: now also J4.A7 (DN1), J4.B7 (DN2)
- net at U5.17 (VCCD): now also C10.2
- net at U5.19 (~RESET): now also R8.2, R9.1
- net VBUS: now reaches U5.20 (VCC)
- net VBUS: now also C8.1, C9.2, J4.A4_B9 (VBUS), J4.B4_A9 (VBUS), R8.1
- net AVR_RX: now reaches U5.5 (RXD)
- net DataEntry_A renamed DPad_Jump
- net DPad_Jump: now also SW48.1; no longer SW42.A
- net DataEntry_B renamed MD_Voice
- net MD_Voice: now also SW49.1; no longer SW42.B
- net Knob1_A renamed MD_Multi
- net MD_Multi: now also SW50.1
- net Knob1_B: no longer names the net of U4.22 (GPA1)
- net Knob2_A: no longer names the net of U4.23 (GPA2)
- net Knob2_B: no longer names the net of U4.24 (GPA3)
- net Knob3_A: no longer names the net of U4.25 (GPA4)
- net Knob3_B: no longer names the net of U4.26 (GPA5)
- net Knob4_A: no longer names the net of U4.27 (GPA6)
- net Knob4_B: no longer names the net of U4.28 (GPA7)
- new net: J4.A5 (CC1), R10.1
- new net: J4.B5 (CC2), R11.1
- new net: D1.2 (A), R12.1
- no-connect marks 102 -> 120
Other:
- note added: "EEPROM"
- note added: "LEDs"
- note added: "USB-UART"
- note added: "User Interace: Data Entry Rotary Knobs"
- note removed: "User Interace: Data Entry Potentiometers"
- moved on the sheet: C1, C2, C3, C4, C5, IC1, J1, J2, J3, R1, R2, R3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

Commit message: lots of ui board routing
Parts:
- added J5: SPI Pins, Connector_PinHeader_2.54mm:PinHeader_1x06_P2.54mm_Vertical, symbol Connector:Conn_01x06_Female
- added R13, R14: 4.7k, Resistor_SMD:R_0805_2012Metric_Pad1.20x1.40mm_HandSolder, symbol Device:R
- added U6: MCP23017_SO (0x24), Package_SO:SOIC-28W_7.5x17.9mm_P1.27mm, symbol Interface_Expansion:MCP23017_SO
- SW1: value Arduino Reset Pusbutton -> Reset
Connections:
- net UART_RX_5V is gone; now on net TX1_D46: J1.8 (Pin_8)
- net UART_TX_5V is gone; now on net RX1_D45: J1.7 (Pin_7)
- net +5V: now also J5.5 (Pin_5), R13.1, R14.2, U6.17 (A2), U6.9 (VDD)
- net D22: now also J5.1 (Pin_1)
- net D25: now also SW42.B
- net D26: now also SW42.A; no longer SW44.A1 (CCW)
- net D28: now also SW44.A1 (CCW); no longer SW46.A1 (CCW)
- net D29: now also SW41.C1 (CW); no longer SW46.C1 (CW)
- net D30: now also SW47.C1 (CW); no longer SW42.A
- net D31: now also SW47.A1 (CCW); no longer SW42.B
- net D32: now also SW45.C1 (CW); no longer SW40.A1 (CCW)
- net D33: now also SW45.A1 (CCW); no longer SW40.C1 (CW)
- net D34: now also SW43.C1 (CW); no longer SW43.A1 (CCW)
- net D35: now also SW43.A1 (CCW); no longer SW43.C1 (CW)
- net D36: now also SW40.C1 (CW); no longer SW45.A1 (CCW)
- net D37: now also SW40.A1 (CCW); no longer SW45.C1 (CW)
- net D38: no longer SW47.A1 (CCW)
- net D39: now also SW41.A1 (CCW); no longer SW47.C1 (CW)
- net D40: now also SW46.C1 (CW); no longer SW41.A1 (CCW)
- net D41: now also SW46.A1 (CCW); no longer SW41.C1 (CW)
- net DPad_Down: now also U3.5 (GPB4); no longer U2.26 (GPA5)
- net DPad_Element: now also U3.8 (GPB7); no longer U3.6 (GPB5)
- net DPad_Jump: now also U3.26 (GPA5); no longer U4.7 (GPB6)
- net DPad_Left: now also U3.1 (GPB0); no longer U2.27 (GPA6)
- net DPad_No: now also U3.2 (GPB1); no longer U3.1 (GPB0)
- net DPad_Operator: now also U3.25 (GPA4); no longer U3.7 (GPB6)
- net DPad_Page_Next: now also U3.7 (GPB6); no longer U3.4 (GPB3)
- net DPad_Right: now also U3.28 (GPA7); no longer U2.28 (GPA7)
- net DPad_Select: now also U3.4 (GPB3); no longer U3.5 (GPB4)
- net DPad_Up: now also U3.6 (GPB5); no longer U2.25 (GPA4)
- net DPad_Yes: now also U3.27 (GPA6); no longer U3.2 (GPB1)
- net FK_Exit: now also U6.22 (GPA1); no longer U4.1 (GPB0)
- net FK_F1: now also U6.2 (GPB1); no longer U3.21 (GPA0)
- net FK_F2: now also U6.3 (GPB2); no longer U3.22 (GPA1)
- net FK_F3: now also U6.4 (GPB3); no longer U3.23 (GPA2)
- net FK_F4: now also U6.5 (GPB4); no longer U3.24 (GPA3)
- net FK_F5: now also U6.6 (GPB5); no longer U3.25 (GPA4)
- net FK_F6: now also U6.7 (GPB6); no longer U3.26 (GPA5)
- net FK_F7: now also U6.8 (GPB7); no longer U3.27 (GPA6)
- net FK_F8: now also U6.21 (GPA0); no longer U3.28 (GPA7)
- net FK_Shift: now also U6.1 (GPB0); no longer U3.8 (GPB7)
- net GND: now also J5.6 (Pin_6), U6.10 (VSS), U6.15 (A0), U6.16 (A1), U6.18 (~RESET~)
- net MD_Copy: now also U4.28 (GPA7); no longer U4.4 (GPB3)
- net MD_EF_Bypass: now also U4.1 (GPB0); no longer U4.6 (GPB5)
- net MD_Edit: now also U4.2 (GPB1); no longer U4.3 (GPB2)
- net MD_Memory: now also U4.26 (GPA5); no longer U4.5 (GPB4)
- net MD_Multi: now also U4.27 (GPA6); no longer U4.21 (GPA0)
- net MD_Utility: now also U4.25 (GPA4); no longer U4.2 (GPB1)
- net MD_Voice: now also U4.3 (GPB2); no longer U4.8 (GPB7)
- net MISO_D50: now also J5.4 (Pin_4)
- net MOSI_D51: now also J5.3 (Pin_3)
- net Numpad_2: now also U2.6 (GPB5); no longer U2.3 (GPB2)
- net Numpad_3: now also U2.27 (GPA6); no longer U2.4 (GPB3)
- net Numpad_4: now also U2.3 (GPB2); no longer U2.5 (GPB4)
- net Numpad_5: now also U2.7 (GPB6); no longer U2.6 (GPB5)
- net Numpad_6: now also U2.26 (GPA5); no longer U2.7 (GPB6)
- net Numpad_7: now also U2.4 (GPB3); no longer U2.8 (GPB7)
- net Numpad_8: now also U2.8 (GPB7); no longer U2.21 (GPA0)
- net Numpad_9: now also U2.25 (GPA4); no longer U2.22 (GPA1)
- net Numpad_Enter: now also U2.28 (GPA7); no longer U2.24 (GPA3)
- net Numpad_Sign: now also U2.5 (GPB4); no longer U2.23 (GPA2)
- net SCK_D52: now also J5.2 (Pin_2)
- net SCL_D21: now also R14.1, U6.12 (SCK)
- net SDA_D20: now also R13.2, U6.13 (SDA)
- no-connect marks 120 -> 133
Other:
- note removed: "User Interace: Multiplexer"
- moved on the sheet: R2, R3, R4, R5, R6, R7, RV3, SW10, SW11, SW12, SW13, SW14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

Commit message: updated footprint for the crystal
Parts:
- Y1: footprint Crystal:Crystal_SMD_2012-2Pin_2.0x1.2mm_HandSoldering -> Crystal:Crystal_SMD_3225-4Pin_3.2x2.5mm_HandSoldering
Changed lines of the file:
@@
 F 0 "Y1" V 5154 4181 50  0000 L CNN
 F 1 "Crystal 16MHz" V 5245 4181 50  0000 L CNN
-F 2 "Crystal:Crystal_SMD_2012-2Pin_2.0x1.2mm_HandSoldering" H 5200 4050 50  0001 C CNN
+F 2 "Crystal:Crystal_SMD_3225-4Pin_3.2x2.5mm_HandSoldering" H 5200 4050 50  0001 C CNN
 F 3 "~" H 5200 4050 50  0001 C CNN
 	1    5200 4050
